Commit message: Change library to dynamixel

File: open_manipulator_x_description_rosbot/urdf/open_manipulator_x.xacro (robot description, xacro)
@@ -248,7 +248,7 @@
         <hardware>
           <plugin>open_manipulator_x_hardware/OpenManipulatorXSystem</plugin>
-          <param name="opencr_id">200</param>
-          <param name="opencr_usb_port">/dev/ttyUSB0</param>
-          <param name="opencr_baud_rate">115200</param>
+          <param name="usb_port">/dev/ttyUSB0</param>
+          <param name="baud_rate">115200</param>
+          <param name="control_period">0.01</param>
           <param name="dxl_joints_profile_acceleration">100</param>
           <param name="dxl_joints_profile_velocity">500</param>
@@ -297,5 +297,5 @@
         <state_interface name="velocity" />
       </joint>
-      <!-- <joint name="${tf_prefix_ext}gripper_right_joint">
+      <joint name="${tf_prefix_ext}gripper_right_joint">
         <param name="mimic">gripper_left_joint</param>
         <param name="multiplier">1</param>
@@ -306,5 +306,5 @@
         <state_interface name="position"/>
         <state_interface name="velocity"/>
-      </joint> -->
+      </joint>
     </ros2_control>
   </xacro:macro>

Commit message: Fix moveit config

File: open_manipulator_x_description_rosbot/urdf/open_manipulator_x.xacro (robot description, xacro)
@@ -21,4 +21,7 @@
       name="meshes_file_direction"
       value="file://$(find ros_components_description)/meshes/open_manipulator_x" />
+    <material name="grey">
+      <color rgba="0.05 0.05 0.05 1.0" />
+    </material>
     <link name="${tf_prefix_ext}link1">
       <visual>
@@ -230,5 +233,5 @@
     </joint>
     <link name="${tf_prefix_ext}end_effector_link">
-      <visual>
+      <!-- <visual>
         <origin xyz="0 0 0" rpy="0 0 0" />
         <geometry>
@@ -236,5 +239,5 @@
         </geometry>
         <material name="red" />
-      </visual>
+      </visual> -->
     </link>
     <ros2_control name="manipulator" type="system">
@@ -297,5 +300,5 @@
         <state_interface name="velocity" />
       </joint>
-      <joint name="${tf_prefix_ext}gripper_right_joint">
+      <!-- <joint name="${tf_prefix_ext}gripper_right_joint">
         <param name="mimic">gripper_left_joint</param>
         <param name="multiplier">1</param>
@@ -306,5 +309,5 @@
         <state_interface name="position"/>
         <state_interface name="velocity"/>
-      </joint>
+      </joint> -->
     </ros2_control>
   </xacro:macro>

Commit message: Fix gripper

File: open_manipulator_x_description_rosbot/urdf/open_manipulator_x.xacro (robot description, xacro)
@@ -300,5 +300,5 @@
         <state_interface name="velocity" />
       </joint>
-      <!-- <joint name="${tf_prefix_ext}gripper_right_joint">
+      <joint name="${tf_prefix_ext}gripper_right_joint">
         <param name="mimic">gripper_left_joint</param>
         <param name="multiplier">1</param>
@@ -309,5 +309,5 @@
         <state_interface name="position"/>
         <state_interface name="velocity"/>
-      </joint> -->
+      </joint>
     </ros2_control>
   </xacro:macro>

Commit message: Add collision enabled parameter to urdf

File: open_manipulator_x_description_rosbot/urdf/open_manipulator_x.xacro (robot description, xacro)
@@ -6,5 +6,8 @@
 -->
 <robot xmlns:xacro="http://www.ros.org/wiki/xacro">
-  <xacro:macro name="open_manipulator_x" params="parent_link xyz rpy tf_prefix:=None use_sim">
+  <xacro:macro name="open_manipulator_x"
+    params="parent_link xyz rpy tf_prefix:=None use_sim collision_enabled:=True">
+    <!-- collision_enabled parameter added due to collisions using visual meshes, which are very
+    heavy and slow down simulation, this parameter allows to easily disable them -->
     <xacro:if value="${tf_prefix == 'None'}">
       <xacro:property name="tf_prefix_ext" value="" />
@@ -32,10 +35,12 @@
         <material name="grey" />
       </visual>
-      <collision>
-        <origin xyz="0 0 0" rpy="0 0 0" />
-        <geometry>
-          <mesh filename="${meshes_file_direction}/link1.stl" scale="0.001 0.001 0.001" />
-        </geometry>
-      </collision>
+      <xacro:if value="${collision_enabled}">
+        <collision>
+          <origin xyz="0 0 0" rpy="0 0 0" />
+          <geometry>
+            <mesh filename="${meshes_file_direction}/link1.stl" scale="0.001 0.001 0.001" />
+          </geometry>
+        </collision>
+      </xacro:if>
       <inertial>
         <origin xyz="3.0876154e-04 0.0000000e+00 -1.2176461e-04" />
@@ -62,10 +67,13 @@
         <material name="grey" />
       </visual>
-      <collision>
-        <origin xyz="0 0 0.019" rpy="0 0 0" />
-        <geometry>
-          <mesh filename="${meshes_file_direction}/link2.stl" scale="0.001 0.001 0.001" />
-        </geometry>
-      </collision>
+      <xacro:if value="${collision_enabled}">
+        <collision>
+          <origin xyz="0 0 0.019" rpy="0 0 0" />
+          <geometry>
+            <mesh
+              filename="${meshes_file_direction}/link2.stl" scale="0.001 0.001 0.001" />
+          </geometry>
+        </collision>
+      </xacro:if>
       <inertial>
         <origin xyz="-3.0184870e-04 5.4043684e-04 ${0.018 + 2.9433464e-02}" />
@@ -92,10 +100,13 @@
         <material name="grey" />
       </visual>
-      <collision>
-        <origin xyz="0 0 0" rpy="0 0 0" />
-        <geometry>
-          <mesh filename="${meshes_file_direction}/link3.stl" scale="0.001 0.001 0.001" />
-        </geometry>
-      </collision>
+      <xacro:if value="${collision_enabled}">
+        <collision>
+          <origin xyz="0 0 0" rpy="0 0 0" />
+          <geometry>
+            <mesh
+              filename="${meshes_file_direction}/link3.stl" scale="0.001 0.001 0.001" />
+          </geometry>
+        </collision>
+      </xacro:if>
       <inertial>
         <origin xyz="1.0308393e-02 3.7743363e-04 1.0170197e-01" />
@@ -122,10 +133,13 @@
         <material name="grey" />
       </visual>
-      <collision>
-        <origin xyz="0 0 0" rpy="0 0 0" />
-        <geometry>
-          <mesh filename="${meshes_file_direction}/link4.stl" scale="0.001 0.001 0.001" />
-        </geometry>
-      </collision>
+      <xacro:if value="${collision_enabled}">
+        <collision>
+          <origin xyz="0 0 0" rpy="0 0 0" />
+          <geometry>
+            <mesh
+              filename="${meshes_file_direction}/link4.stl" scale="0.001 0.001 0.001" />
+          </geometry>
+        </collision>
+      </xacro:if>
       <inertial>
         <origin xyz="9.0909590e-02 3.8929816e-04 2.2413279e-04" />
@@ -152,10 +166,13 @@
         <material name="grey" />
       </visual>
-      <collision>
-        <origin xyz="0 0 0" rpy="0 0 0" />
-        <geometry>
-          <mesh filename="${meshes_file_direction}/link5.stl" scale="0.001 0.001 0.001" />
-        </geometry>
-      </collision>
+      <xacro:if value="${collision_enabled}">
+        <collision>
+          <origin xyz="0 0 0" rpy="0 0 0" />
+          <geometry>
+            <mesh
+              filename="${meshes_file_direction}/link5.stl" scale="0.001 0.001 0.001" />
+          </geometry>
+        </collision>
+      </xacro:if>
       <inertial>
         <origin xyz="4.4206755e-02 3.6839985e-07 8.9142216e-03" />
@@ -182,10 +199,13 @@
         <material name="grey" />
       </visual>
-      <collision>
-        <origin xyz="0 0 0" rpy="0 0 0" />
-        <geometry>
-          <mesh filename="${meshes_file_direction}/gripper_left_palm.stl" scale="0.001 0.001 0.001" />
-        </geometry>
-      </collision>
+      <xacro:if value="${collision_enabled}">
+        <collision>
+          <origin xyz="0 0 0" rpy="0 0 0" />
+          <geometry>
+            <mesh
+              filename="${meshes_file_direction}/gripper_left_palm.stl" scale="0.001 0.001 0.001" />
+          </geometry>
+        </collision>
+      </xacro:if>
       <inertial>
         <origin xyz="0 0 0" />
@@ -213,10 +233,13 @@
         <material name="grey" />
       </visual>
-      <collision>
-        <origin xyz="0 0 0" rpy="0 0 0" />
-        <geometry>
-          <mesh filename="${meshes_file_direction}/gripper_right_palm.stl" scale="0.001 0.001 0.001" />
-        </geometry>
-      </collision>
+      <xacro:if value="${collision_enabled}">
+        <collision>
+          <origin xyz="0 0 0" rpy="0 0 0" />
+          <geometry>
+            <mesh
+              filename="${meshes_file_direction}/gripper_right_palm.stl" scale="0.001 0.001 0.001" />
+          </geometry>
+        </collision>
+      </xacro:if>
       <inertial>
         <origin xyz="0 0 0" />
@@ -236,5 +259,6 @@
         <origin xyz="0 0 0" rpy="0 0 0" />
         <geometry>
-          <box size="0.01 0.01 0.01" />
+          <box
+      size="0.01 0.01 0.01" />
         </geometry>
         <material name="red" />
@@ -306,6 +330,6 @@
           <param name="max">0.019</param>
         </command_interface>
-        <state_interface name="position"/>
-        <state_interface name="velocity"/>
+        <state_interface name="position" />
+        <state_interface name="velocity" />
       </joint>
     </ros2_control>

Commit message: Adjust joint limits

File: open_manipulator_x_description_rosbot/urdf/open_manipulator_x.xacro (robot description, xacro)
@@ -7,5 +7,5 @@
 <robot xmlns:xacro="http://www.ros.org/wiki/xacro">
   <xacro:macro name="open_manipulator_x"
-    params="parent_link xyz rpy tf_prefix:=None use_sim collision_enabled:=True">
+    params="parent_link xyz rpy tf_prefix:=None use_sim collision_enabled:=true">
     <!-- collision_enabled parameter added due to collisions using visual meshes, which are very
     heavy and slow down simulation, this parameter allows to easily disable them -->
@@ -56,5 +56,5 @@
       <origin xyz="0.012 0.0 0.017" rpy="0 0 0" />
       <axis xyz="0 0 1" />
-      <limit velocity="4.8" effort="1" lower="${-pi*0.9}" upper="${pi*0.9}" />
+      <limit velocity="4.8" effort="1" lower="${-pi*205./180.}" upper="${pi*205./180.}" />
       <dynamics damping="0.1" />
     </joint>
@@ -122,5 +122,5 @@
       <origin xyz="0.024 0 0.128" rpy="0 0 0" />
       <axis xyz="0 1 0" />
-      <limit velocity="4.8" effort="1" lower="${-pi*0.3}" upper="${pi*0.44}" />
+      <limit velocity="4.8" effort="1" lower="${-pi*0.5}" upper="${pi*0.44}" />
       <dynamics damping="0.1" />
     </joint>
@@ -155,5 +155,5 @@
       <origin xyz="0.124 0.0 0.0" rpy="0 0 0" />
       <axis xyz="0 1 0" />
-      <limit velocity="4.8" effort="1" lower="${-pi*0.57}" upper="${pi*0.65}" />
+      <limit velocity="4.8" effort="1" lower="${-pi*0.55}" upper="${pi*0.65}" />
       <dynamics damping="0.1" />
     </joint>
