Commit message: Change limits of joint1

File: open_manipulator_x_description/urdf/open_manipulator_x_macro.urdf.xacro (robot description, xacro)
@@ -52,5 +52,6 @@
       <origin xyz="0.012 0.0 0.017" rpy="0 0 0" />
       <axis xyz="0 0 1" />
-      <limit velocity="${velocity_limit}" effort="${effort_limit}" lower="${-pi*205./180.}" upper="${pi*205./180.}" />
+      <!-- Joint1 motion is limited only by length of the cable -->
+      <limit velocity="${velocity_limit}" effort="${effort_limit}" lower="${-pi*135./180.}" upper="${pi*340./180.}" />
       <dynamics damping="${damping}" />
     </joint>

Commit message: Add arguments with joint1 limits

File: open_manipulator_x_description/urdf/open_manipulator_x_macro.urdf.xacro (robot description, xacro)
@@ -3,5 +3,5 @@
 <robot xmlns:xacro="http://www.ros.org/wiki/xacro">
   <xacro:macro name="open_manipulator_x"
-    params="parent_link xyz rpy tf_prefix:=None use_sim collision_enabled:=true usb_port:=/dev/ttyUSB0 baud_rate:=115200">
+  params="parent_link xyz rpy tf_prefix:=None use_sim collision_enabled:=true usb_port:=/dev/ttyUSB0 baud_rate:=115200 joint1_limit_min:=-2.356 joint1_limit_max:=5.934">
     <!-- collision_enabled parameter added due to collisions using visual meshes, which are very
     heavy and slow down simulation, this parameter allows to easily disable them -->
@@ -53,5 +53,5 @@
       <axis xyz="0 0 1" />
       <!-- Joint1 motion is limited only by length of the cable -->
-      <limit velocity="${velocity_limit}" effort="${effort_limit}" lower="${-pi*135./180.}" upper="${pi*340./180.}" />
+      <limit velocity="${velocity_limit}" effort="${effort_limit}" lower="${joint1_limit_min}" upper="${joint1_limit_max}" />
       <dynamics damping="${damping}" />
     </joint>

Commit message: Update formatting and style of urdf

File: open_manipulator_x_description/urdf/open_manipulator_x_macro.urdf.xacro (robot description, xacro)
@@ -3,5 +3,11 @@
 <robot xmlns:xacro="http://www.ros.org/wiki/xacro">
   <xacro:macro name="open_manipulator_x"
-  params="parent_link xyz rpy tf_prefix:=None use_sim collision_enabled:=true usb_port:=/dev/ttyUSB0 baud_rate:=115200 joint1_limit_min:=-2.356 joint1_limit_max:=5.934">
+    params="parent_link xyz rpy
+            tf_prefix:=None
+            use_sim collision_enabled:=true
+            usb_port:=/dev/ttyUSB0
+            baud_rate:=115200
+            joint1_limit_min:=-2.356
+            joint1_limit_max:=5.934">
     <!-- collision_enabled parameter added due to collisions using visual meshes, which are very
     heavy and slow down simulation, this parameter allows to easily disable them -->
@@ -25,15 +31,17 @@
     <link name="${tf_prefix_ext}link1">
       <visual>
-        <origin xyz="0 0 0" rpy="0 0 0" />
-        <geometry>
-          <mesh filename="file://$(find open_manipulator_x_description)/meshes/link1.stl" scale="0.001 0.001 0.001" />
-        </geometry>
-        <material name="grey" />
-      </visual>
-      <xacro:if value="${collision_enabled}">
-        <collision>
-          <origin xyz="0 0 0" rpy="0 0 0" />
-          <geometry>
-            <mesh filename="file://$(find open_manipulator_x_description)/meshes/link1.stl" scale="0.001 0.001 0.001" />
+        <origin xyz="0.0 0.0 0.0" rpy="0.0 0.0 0.0" />
+        <geometry>
+          <mesh filename="file://$(find open_manipulator_x_description)/meshes/link1.stl"
+            scale="0.001 0.001 0.001" />
+        </geometry>
+        <material name="grey" />
+      </visual>
+      <xacro:if value="${collision_enabled}">
+        <collision>
+          <origin xyz="0.0 0.0 0.0" rpy="0.0 0.0 0.0" />
+          <geometry>
+            <mesh filename="file://$(find open_manipulator_x_description)/meshes/link1.stl"
+              scale="0.001 0.001 0.001" />
           </geometry>
         </collision>
@@ -42,7 +50,7 @@
         <origin xyz="3.0876154e-04 0.0000000e+00 -1.2176461e-04" />
         <mass value="7.9119962e-02" />
-        <inertia ixx="1.2505234e-05" ixy="0.0" ixz="-1.7855208e-07"
-          iyy="2.1898364e-05" iyz="0.0"
-          izz="1.9267361e-05" />
+        <inertia ixx="1.2505234e-05" ixy="0.0"           ixz="-1.7855208e-07"
+                                     iyy="2.1898364e-05" iyz="0.0"
+                                                         izz="1.9267361e-05" />
       </inertial>
     </link>
@@ -50,24 +58,27 @@
       <parent link="${tf_prefix_ext}link1" />
       <child link="${tf_prefix_ext}link2" />
-      <origin xyz="0.012 0.0 0.017" rpy="0 0 0" />
+      <origin xyz="0.012 0.0 0.017" rpy="0.0 0.0 0.0" />
       <axis xyz="0 0 1" />
       <!-- Joint1 motion is limited only by length of the cable -->
-      <limit velocity="${velocity_limit}" effort="${effort_limit}" lower="${joint1_limit_min}" upper="${joint1_limit_max}" />
+      <limit velocity="${velocity_limit}" effort="${effort_limit}" lower="${joint1_limit_min}"
+        upper="${joint1_limit_max}" />
       <dynamics damping="${damping}" />
     </joint>
     <link name="${tf_prefix_ext}link2">
       <visual>
-        <origin xyz="0 0 0.019" rpy="0 0 0" />
-        <geometry>
-          <mesh filename="file://$(find open_manipulator_x_description)/meshes/link2.stl" scale="0.001 0.001 0.001" />
-        </geometry>
-        <material name="grey" />
-      </visual>
-      <xacro:if value="${collision_enabled}">
-        <collision>
-          <origin xyz="0 0 0.019" rpy="0 0 0" />
-          <geometry>
-            <mesh
-              filename="file://$(find open_manipulator_x_description)/meshes/link2.stl" scale="0.001 0.001 0.001" />
+        <origin xyz="0.0 0.0 0.019" rpy="0.0 0.0 0.0" />
+        <geometry>
+          <mesh filename="file://$(find open_manipulator_x_description)/meshes/link2.stl"
+            scale="0.001 0.001 0.001" />
+        </geometry>
+        <material name="grey" />
+      </visual>
+      <xacro:if value="${collision_enabled}">
+        <collision>
+          <origin xyz="0.0 0.0 0.019" rpy="0.0 0.0 0.0" />
+          <geometry>
+            <mesh
+              filename="file://$(find open_manipulator_x_description)/meshes/link2.stl"
+              scale="0.001 0.001 0.001" />
           </geometry>
         </collision>
@@ -77,6 +88,6 @@
         <mass value="9.8406837e-02" />
         <inertia ixx="3.4543422e-05" ixy="-1.6031095e-08" ixz="-3.8375155e-07"
-          iyy="3.2689329e-05" iyz="2.8511935e-08"
-          izz="1.8850320e-05" />
+                                     iyy="3.2689329e-05"  iyz="2.8511935e-08"
+                                                          izz="1.8850320e-05" />
       </inertial>
     </link>
@@ -84,23 +95,26 @@
       <parent link="${tf_prefix_ext}link2" />
       <child link="${tf_prefix_ext}link3" />
-      <origin xyz="0.0 0.0 0.0595" rpy="0 0 0" />
+      <origin xyz="0.0 0.0 0.0595" rpy="0.0 0.0 0.0" />
       <axis xyz="0 1 0" />
-      <limit velocity="${velocity_limit}" effort="${effort_limit}" lower="${-pi*0.57}" upper="${pi*0.5}" />
+      <limit velocity="${velocity_limit}" effort="${effort_limit}" lower="${-pi*0.57}"
+        upper="${pi*0.5}" />
       <dynamics damping="${damping}" />
     </joint>
     <link name="${tf_prefix_ext}link3">
       <visual>
-        <origin xyz="0 0 0" rpy="0 0 0" />
-        <geometry>
-          <mesh filename="file://$(find open_manipulator_x_description)/meshes/link3.stl" scale="0.001 0.001 0.001" />
-        </geometry>
-        <material name="grey" />
-      </visual>
-      <xacro:if value="${collision_enabled}">
-        <collision>
-          <origin xyz="0 0 0" rpy="0 0 0" />
-          <geometry>
-            <mesh
-              filename="file://$(find open_manipulator_x_description)/meshes/link3.stl" scale="0.001 0.001 0.001" />
+        <origin xyz="0.0 0.0 0.0" rpy="0.0 0.0 0.0" />
+        <geometry>
+          <mesh filename="file://$(find open_manipulator_x_description)/meshes/link3.stl"
+            scale="0.001 0.001 0.001" />
+        </geometry>
+        <material name="grey" />
+      </visual>
+      <xacro:if value="${collision_enabled}">
+        <collision>
+          <origin xyz="0.0 0.0 0.0" rpy="0.0 0.0 0.0" />
+          <geometry>
+            <mesh
+              filename="file://$(find open_manipulator_x_description)/meshes/link3.stl"
+              scale="0.001 0.001 0.001" />
           </geometry>
         </collision>
@@ -110,6 +124,6 @@
         <mass value="1.3850917e-01" />
         <inertia ixx="3.3055381e-04" ixy="-9.7940978e-08" ixz="-3.8505711e-05"
-          iyy="3.4290447e-04" iyz="-1.5717516e-06"
-          izz="6.0346498e-05" />
+                                     iyy="3.4290447e-04"  iyz="-1.5717516e-06"
+                                                          izz="6.0346498e-05" />
       </inertial>
     </link>
@@ -117,23 +131,26 @@
       <parent link="${tf_prefix_ext}link3" />
       <child link="${tf_prefix_ext}link4" />
-      <origin xyz="0.024 0 0.128" rpy="0 0 0" />
+      <origin xyz="0.024 0.0 0.128" rpy="0.0 0.0 0.0" />
       <axis xyz="0 1 0" />
-      <limit velocity="${velocity_limit}" effort="${effort_limit}" lower="${-pi*0.5}" upper="${pi*0.44}" />
+      <limit velocity="${velocity_limit}" effort="${effort_limit}" lower="${-pi*0.5}"
+        upper="${pi*0.44}" />
       <dynamics damping="${damping}" />
     </joint>
     <link name="${tf_prefix_ext}link4">
       <visual>
-        <origin xyz="0 0 0" rpy="0 0 0" />
-        <geometry>
-          <mesh filename="file://$(find open_manipulator_x_description)/meshes/link4.stl" scale="0.001 0.001 0.001" />
-        </geometry>
-        <material name="grey" />
-      </visual>
-      <xacro:if value="${collision_enabled}">
-        <collision>
-          <origin xyz="0 0 0" rpy="0 0 0" />
-          <geometry>
-            <mesh
-              filename="file://$(find open_manipulator_x_description)/meshes/link4.stl" scale="0.001 0.001 0.001" />
+        <origin xyz="0.0 0.0 0.0" rpy="0.0 0.0 0.0" />
+        <geometry>
+          <mesh filename="file://$(find open_manipulator_x_description)/meshes/link4.stl"
+            scale="0.001 0.001 0.001" />
+        </geometry>
+        <material name="grey" />
+      </visual>
+      <xacro:if value="${collision_enabled}">
+        <collision>
+          <origin xyz="0.0 0.0 0.0" rpy="0.0 0.0 0.0" />
+          <geometry>
+            <mesh
+              filename="file://$(find open_manipulator_x_description)/meshes/link4.stl"
+              scale="0.001 0.001 0.001" />
           </geometry>
         </collision>
@@ -143,6 +160,6 @@
         <mass value="1.3274562e-01" />
         <inertia ixx="3.0654178e-05" ixy="-1.2764155e-06" ixz="-2.6874417e-07"
-          iyy="2.4230292e-04" iyz="1.1559550e-08"
-          izz="2.5155057e-04" />
+                                     iyy="2.4230292e-04"  iyz="1.1559550e-08"
+                                                          izz="2.5155057e-04" />
       </inertial>
     </link>
@@ -150,23 +167,26 @@
       <parent link="${tf_prefix_ext}link4" />
       <child link="${tf_prefix_ext}link5" />
-      <origin xyz="0.124 0.0 0.0" rpy="0 0 0" />
+      <origin xyz="0.124 0.0 0.0" rpy="0.0 0.0 0.0" />
       <axis xyz="0 1 0" />
-      <limit velocity="${velocity_limit}" effort="${effort_limit}" lower="${-pi*0.55}" upper="${pi*0.65}" />
+      <limit velocity="${velocity_limit}" effort="${effort_limit}" lower="${-pi*0.55}"
+        upper="${pi*0.65}" />
       <dynamics damping="${damping}" />
     </joint>
     <link name="${tf_prefix_ext}link5">
       <visual>
-        <origin xyz="0 0 0" rpy="0 0 0" />
-        <geometry>
-          <mesh filename="file://$(find open_manipulator_x_description)/meshes/link5.stl" scale="0.001 0.001 0.001" />
-        </geometry>
-        <material name="grey" />
-      </visual>
-      <xacro:if value="${collision_enabled}">
-        <collision>
-          <origin xyz="0 0 0" rpy="0 0 0" />
-          <geometry>
-            <mesh
-              filename="file://$(find open_manipulator_x_description)/meshes/link5.stl" scale="0.001 0.001 0.001" />
+        <origin xyz="0.0 0.0 0.0" rpy="0.0 0.0 0.0" />
+        <geometry>
+          <mesh filename="file://$(find open_manipulator_x_description)/meshes/link5.stl"
+            scale="0.001 0.001 0.001" />
+        </geometry>
+        <material name="grey" />
+      </visual>
+      <xacro:if value="${collision_enabled}">
+        <collision>
+          <origin xyz="0.0 0.0 0.0" rpy="0.0 0.0 0.0" />
+          <geometry>
+            <mesh
+              filename="file://$(find open_manipulator_x_description)/meshes/link5.stl"
+              scale="0.001 0.001 0.001" />
           </geometry>
         </collision>
@@ -175,7 +195,7 @@
         <origin xyz="4.4206755e-02 3.6839985e-07 8.9142216e-03" />
         <mass value="1.4327573e-01" />
-        <inertia ixx="8.0870749e-05" ixy="0.0" ixz="-1.0157896e-06"
-          iyy="7.5980465e-05" iyz="0.0"
-          izz="9.3127351e-05" />
+        <inertia ixx="8.0870749e-05" ixy="0.0"           ixz="-1.0157896e-06"
+                                     iyy="7.5980465e-05" iyz="0.0"
+                                                         izz="9.3127351e-05" />
       </inertial>
     </link>
@@ -183,5 +203,5 @@
       <parent link="${tf_prefix_ext}link5" />
       <child link="${tf_prefix_ext}gripper_left_link" />
-      <origin xyz="0.0817 0.021 0.0" rpy="0 0 0" />
+      <origin xyz="0.0817 0.021 0.0" rpy="0.0 0.0 0.0" />
       <axis xyz="0 1 0" />
       <limit velocity="${velocity_limit}" effort="${effort_limit}" lower="-0.010" upper="0.019" />
@@ -190,25 +210,28 @@
     <link name="${tf_prefix_ext}gripper_left_link">
       <visual>
-        <origin xyz="0 0 0" rpy="0 0 0" />
-        <geometry>
-          <mesh filename="file://$(find open_manipulator_x_description)/meshes/gripper_left_palm.stl" scale="0.001 0.001 0.001" />
-        </geometry>
-        <material name="grey" />
-      </visual>
-      <xacro:if value="${collision_enabled}">
-        <collision>
-          <origin xyz="0 0 0" rpy="0 0 0" />
-          <geometry>
-            <mesh
-              filename="file://$(find open_manipulator_x_description)/meshes/gripper_left_palm.stl" scale="0.001 0.001 0.001" />
-          </geometry>
-        </collision>
-      </xacro:if>
-      <inertial>
-        <origin xyz="0 0 0" />
+        <origin xyz="0.0 0.0 0.0" rpy="0.0 0.0 0.0" />
+        <geometry>
+          <mesh
+            filename="file://$(find open_manipulator_x_description)/meshes/gripper_left_palm.stl"
+            scale="0.001 0.001 0.001" />
+        </geometry>
+        <material name="grey" />
+      </visual>
+      <xacro:if value="${collision_enabled}">
+        <collision>
+          <origin xyz="0.0 0.0 0.0" rpy="0.0 0.0 0.0" />
+          <geometry>
+            <mesh
+              filename="file://$(find open_manipulator_x_description)/meshes/gripper_left_palm.stl"
+              scale="0.001 0.001 0.001" />
+          </geometry>
+        </collision>
+      </xacro:if>
+      <inertial>
+        <origin xyz="0.0 0.0 0.0" />
         <mass value="1.0e-03" />
-        <inertia ixx="1.0e-06" ixy="0.0" ixz="0.0"
-          iyy="1.0e-06" iyz="0.0"
-          izz="1.0e-06" />
+        <inertia ixx="1.0e-06" ixy="0.0"     ixz="0.0"
+                               iyy="1.0e-06" iyz="0.0"
+                                             izz="1.0e-06" />
       </inertial>
     </link>
@@ -216,5 +239,5 @@
       <parent link="${tf_prefix_ext}link5" />
       <child link="${tf_prefix_ext}gripper_right_link" />
-      <origin xyz="0.0817 -0.021 0" rpy="0 0 0" />
+      <origin xyz="0.0817 -0.021 0.0" rpy="0.0 0.0 0.0" />
       <axis xyz="0 -1 0" />
       <limit velocity="${velocity_limit}" effort="${effort_limit}" lower="-0.010" upper="0.019" />
@@ -224,16 +247,19 @@
     <link name="${tf_prefix_ext}gripper_right_link">
       <visual>
-        <origin xyz="0 0 0" rpy="0 0 0" />
-        <geometry>
-          <mesh filename="file://$(find open_manipulator_x_description)/meshes/gripper_right_palm.stl" scale="0.001 0.001 0.001" />
-        </geometry>
-        <material name="grey" />
-      </visual>
-      <xacro:if value="${collision_enabled}">
-        <collision>
-          <origin xyz="0 0 0" rpy="0 0 0" />
-          <geometry>
-            <mesh
-              filename="file://$(find open_manipulator_x_description)/meshes/gripper_right_palm.stl" scale="0.001 0.001 0.001" />
+        <origin xyz="0.0 0.0 0.0" rpy="0.0 0.0 0.0" />
+        <geometry>
+          <mesh
+            filename="file://$(find open_manipulator_x_description)/meshes/gripper_right_palm.stl"
+            scale="0.001 0.001 0.001" />
+        </geometry>
+        <material name="grey" />
+      </visual>
+      <xacro:if value="${collision_enabled}">
+        <collision>
+          <origin xyz="0.0 0.0 0.0" rpy="0.0 0.0 0.0" />
+          <geometry>
+            <mesh
+              filename="file://$(find open_manipulator_x_description)/meshes/gripper_right_palm.stl"
+              scale="0.001 0.001 0.001" />
           </geometry>
         </collision>
@@ -242,7 +268,7 @@
         <origin xyz="0 0 0" />
         <mass value="1.0e-03" />
-        <inertia ixx="1.0e-06" ixy="0.0" ixz="0.0"
-          iyy="1.0e-06" iyz="0.0"
-          izz="1.0e-06" />
+        <inertia ixx="1.0e-06" ixy="0.0"     ixz="0.0"
+                               iyy="1.0e-06" iyz="0.0"
+                                             izz="1.0e-06" />
       </inertial>
     </link>
@@ -250,5 +276,5 @@
       <parent link="${tf_prefix_ext}link5" />
       <child link="${tf_prefix_ext}end_effector_link" />
-      <origin xyz="0.126 0.0 0.0" rpy="0 0 0" />
+      <origin xyz="0.126 0.0 0.0" rpy="0.0 0.0 0.0" />
     </joint>
     <link name="${tf_prefix_ext}end_effector_link" />
