Commit message: Use package in urdf

File: open_manipulator_x_description/urdf/open_manipulator_x_macro.urdf.xacro (robot description, xacro)
@@ -38,14 +38,14 @@
         <origin xyz="0.0 0.0 0.0" rpy="0.0 0.0 0.0" />
         <geometry>
-          <mesh filename="file://$(find open_manipulator_x_description)/meshes/link1.stl"
-            scale="0.001 0.001 0.001" />
-        </geometry>
-        <material name="grey" />
-      </visual>
-      <xacro:if value="${collision_enabled}">
-        <collision>
-          <origin xyz="0.0 0.0 0.0" rpy="0.0 0.0 0.0" />
-          <geometry>
-            <mesh filename="file://$(find open_manipulator_x_description)/meshes/link1.stl"
+          <mesh filename="package://open_manipulator_x_description/meshes/link1.stl"
+            scale="0.001 0.001 0.001" />
+        </geometry>
+        <material name="grey" />
+      </visual>
+      <xacro:if value="${collision_enabled}">
+        <collision>
+          <origin xyz="0.0 0.0 0.0" rpy="0.0 0.0 0.0" />
+          <geometry>
+            <mesh filename="package://open_manipulator_x_description/meshes/link1.stl"
               scale="0.001 0.001 0.001" />
           </geometry>
@@ -74,5 +74,5 @@
         <origin xyz="0.0 0.0 0.019" rpy="0.0 0.0 0.0" />
         <geometry>
-          <mesh filename="file://$(find open_manipulator_x_description)/meshes/link2.stl"
+          <mesh filename="package://open_manipulator_x_description/meshes/link2.stl"
             scale="0.001 0.001 0.001" />
         </geometry>
@@ -84,5 +84,5 @@
           <geometry>
             <mesh
-              filename="file://$(find open_manipulator_x_description)/meshes/link2.stl"
+              filename="package://open_manipulator_x_description/meshes/link2.stl"
               scale="0.001 0.001 0.001" />
           </geometry>
@@ -110,15 +110,15 @@
         <origin xyz="0.0 0.0 0.0" rpy="0.0 0.0 0.0" />
         <geometry>
-          <mesh filename="file://$(find open_manipulator_x_description)/meshes/link3.stl"
-            scale="0.001 0.001 0.001" />
-        </geometry>
-        <material name="grey" />
-      </visual>
-      <xacro:if value="${collision_enabled}">
-        <collision>
-          <origin xyz="0.0 0.0 0.0" rpy="0.0 0.0 0.0" />
-          <geometry>
-            <mesh
-              filename="file://$(find open_manipulator_x_description)/meshes/link3.stl"
+          <mesh filename="package://open_manipulator_x_description/meshes/link3.stl"
+            scale="0.001 0.001 0.001" />
+        </geometry>
+        <material name="grey" />
+      </visual>
+      <xacro:if value="${collision_enabled}">
+        <collision>
+          <origin xyz="0.0 0.0 0.0" rpy="0.0 0.0 0.0" />
+          <geometry>
+            <mesh
+              filename="package://open_manipulator_x_description/meshes/link3.stl"
               scale="0.001 0.001 0.001" />
           </geometry>
@@ -146,15 +146,15 @@
         <origin xyz="0.0 0.0 0.0" rpy="0.0 0.0 0.0" />
         <geometry>
-          <mesh filename="file://$(find open_manipulator_x_description)/meshes/link4.stl"
-            scale="0.001 0.001 0.001" />
-        </geometry>
-        <material name="grey" />
-      </visual>
-      <xacro:if value="${collision_enabled}">
-        <collision>
-          <origin xyz="0.0 0.0 0.0" rpy="0.0 0.0 0.0" />
-          <geometry>
-            <mesh
-              filename="file://$(find open_manipulator_x_description)/meshes/link4.stl"
+          <mesh filename="package://open_manipulator_x_description/meshes/link4.stl"
+            scale="0.001 0.001 0.001" />
+        </geometry>
+        <material name="grey" />
+      </visual>
+      <xacro:if value="${collision_enabled}">
+        <collision>
+          <origin xyz="0.0 0.0 0.0" rpy="0.0 0.0 0.0" />
+          <geometry>
+            <mesh
+              filename="package://open_manipulator_x_description/meshes/link4.stl"
               scale="0.001 0.001 0.001" />
           </geometry>
@@ -182,15 +182,15 @@
         <origin xyz="0.0 0.0 0.0" rpy="0.0 0.0 0.0" />
         <geometry>
-          <mesh filename="file://$(find open_manipulator_x_description)/meshes/link5.stl"
-            scale="0.001 0.001 0.001" />
-        </geometry>
-        <material name="grey" />
-      </visual>
-      <xacro:if value="${collision_enabled}">
-        <collision>
-          <origin xyz="0.0 0.0 0.0" rpy="0.0 0.0 0.0" />
-          <geometry>
-            <mesh
-              filename="file://$(find open_manipulator_x_description)/meshes/link5.stl"
+          <mesh filename="package://open_manipulator_x_description/meshes/link5.stl"
+            scale="0.001 0.001 0.001" />
+        </geometry>
+        <material name="grey" />
+      </visual>
+      <xacro:if value="${collision_enabled}">
+        <collision>
+          <origin xyz="0.0 0.0 0.0" rpy="0.0 0.0 0.0" />
+          <geometry>
+            <mesh
+              filename="package://open_manipulator_x_description/meshes/link5.stl"
               scale="0.001 0.001 0.001" />
           </geometry>
@@ -218,15 +218,15 @@
         <geometry>
           <mesh
-            filename="file://$(find open_manipulator_x_description)/meshes/gripper_left_palm.stl"
-            scale="0.001 0.001 0.001" />
-        </geometry>
-        <material name="grey" />
-      </visual>
-      <xacro:if value="${collision_enabled}">
-        <collision>
-          <origin xyz="0.0 0.0 0.0" rpy="0.0 0.0 0.0" />
-          <geometry>
-            <mesh
-              filename="file://$(find open_manipulator_x_description)/meshes/gripper_left_palm.stl"
+            filename="package://open_manipulator_x_description/meshes/gripper_left_palm.stl"
+            scale="0.001 0.001 0.001" />
+        </geometry>
+        <material name="grey" />
+      </visual>
+      <xacro:if value="${collision_enabled}">
+        <collision>
+          <origin xyz="0.0 0.0 0.0" rpy="0.0 0.0 0.0" />
+          <geometry>
+            <mesh
+              filename="package://open_manipulator_x_description/meshes/gripper_left_palm.stl"
               scale="0.001 0.001 0.001" />
           </geometry>
@@ -255,15 +255,15 @@
         <geometry>
           <mesh
-            filename="file://$(find open_manipulator_x_description)/meshes/gripper_right_palm.stl"
-            scale="0.001 0.001 0.001" />
-        </geometry>
-        <material name="grey" />
-      </visual>
-      <xacro:if value="${collision_enabled}">
-        <collision>
-          <origin xyz="0.0 0.0 0.0" rpy="0.0 0.0 0.0" />
-          <geometry>
-            <mesh
-              filename="file://$(find open_manipulator_x_description)/meshes/gripper_right_palm.stl"
+            filename="package://open_manipulator_x_description/meshes/gripper_right_palm.stl"
+            scale="0.001 0.001 0.001" />
+        </geometry>
+        <material name="grey" />
+      </visual>
+      <xacro:if value="${collision_enabled}">
+        <collision>
+          <origin xyz="0.0 0.0 0.0" rpy="0.0 0.0 0.0" />
+          <geometry>
+            <mesh
+              filename="package://open_manipulator_x_description/meshes/gripper_right_palm.stl"
               scale="0.001 0.001 0.001" />
           </geometry>

Commit message: Simplify urdf

File: open_manipulator_x_description/urdf/open_manipulator_x_macro.urdf.xacro (robot description, xacro)
@@ -4,5 +4,4 @@
   <xacro:macro name="open_manipulator_x"
     params="parent_link xyz rpy
-            tf_prefix:=None
             use_sim collision_enabled:=true
             usb_port:=/dev/ttyUSB0
@@ -17,10 +16,4 @@
     <!-- collision_enabled parameter added due to collisions using visual meshes, which are very
     heavy and slow down simulation, this parameter allows to easily disable them -->
-    <xacro:if value="${tf_prefix == 'None'}">
-      <xacro:property name="tf_prefix_ext" value="" />
-    </xacro:if>
-    <xacro:unless value="${tf_prefix == 'None'}">
-      <xacro:property name="tf_prefix_ext" value="${tf_prefix}_" />
-    </xacro:unless>
     <material name="grey">
       <color rgba="0.05 0.05 0.05 1.0" />
@@ -29,10 +22,10 @@
     <xacro:property name="velocity_limit" value="4.8" />
     <xacro:property name="damping" value="0.1" />
-    <joint name="${parent_link}_to_${tf_prefix_ext}link1" type="fixed">
+    <joint name="${parent_link}_to_link1" type="fixed">
       <origin xyz="${xyz}" rpy="${rpy}" />
       <parent link="${parent_link}" />
-      <child link="${tf_prefix_ext}link1" />
-    </joint>
-    <link name="${tf_prefix_ext}link1">
+      <child link="link1" />
+    </joint>
+    <link name="link1">
       <visual>
         <origin xyz="0.0 0.0 0.0" rpy="0.0 0.0 0.0" />
@@ -60,7 +53,7 @@
       </inertial>
     </link>
-    <joint name="${tf_prefix_ext}joint1" type="revolute">
-      <parent link="${tf_prefix_ext}link1" />
-      <child link="${tf_prefix_ext}link2" />
+    <joint name="joint1" type="revolute">
+      <parent link="link1" />
+      <child link="link2" />
       <origin xyz="0.012 0.0 0.017" rpy="0.0 0.0 0.0" />
       <axis xyz="0 0 1" />
@@ -70,5 +63,5 @@
       <dynamics damping="${damping}" />
     </joint>
-    <link name="${tf_prefix_ext}link2">
+    <link name="link2">
       <visual>
         <origin xyz="0.0 0.0 0.019" rpy="0.0 0.0 0.0" />
@@ -97,7 +90,7 @@
       </inertial>
     </link>
-    <joint name="${tf_prefix_ext}joint2" type="revolute">
-      <parent link="${tf_prefix_ext}link2" />
-      <child link="${tf_prefix_ext}link3" />
+    <joint name="joint2" type="revolute">
+      <parent link="link2" />
+      <child link="link3" />
       <origin xyz="0.0 0.0 0.0595" rpy="0.0 0.0 0.0" />
       <axis xyz="0 1 0" />
@@ -106,5 +99,5 @@
       <dynamics damping="${damping}" />
     </joint>
-    <link name="${tf_prefix_ext}link3">
+    <link name="link3">
       <visual>
         <origin xyz="0.0 0.0 0.0" rpy="0.0 0.0 0.0" />
@@ -133,7 +126,7 @@
       </inertial>
     </link>
-    <joint name="${tf_prefix_ext}joint3" type="revolute">
-      <parent link="${tf_prefix_ext}link3" />
-      <child link="${tf_prefix_ext}link4" />
+    <joint name="joint3" type="revolute">
+      <parent link="link3" />
+      <child link="link4" />
       <origin xyz="0.024 0.0 0.128" rpy="0.0 0.0 0.0" />
       <axis xyz="0 1 0" />
@@ -142,5 +135,5 @@
       <dynamics damping="${damping}" />
     </joint>
-    <link name="${tf_prefix_ext}link4">
+    <link name="link4">
       <visual>
         <origin xyz="0.0 0.0 0.0" rpy="0.0 0.0 0.0" />
@@ -169,7 +162,7 @@
       </inertial>
     </link>
-    <joint name="${tf_prefix_ext}joint4" type="revolute">
-      <parent link="${tf_prefix_ext}link4" />
-      <child link="${tf_prefix_ext}link5" />
+    <joint name="joint4" type="revolute">
+      <parent link="link4" />
+      <child link="link5" />
       <origin xyz="0.124 0.0 0.0" rpy="0.0 0.0 0.0" />
       <axis xyz="0 1 0" />
@@ -178,5 +171,5 @@
       <dynamics damping="${damping}" />
     </joint>
-    <link name="${tf_prefix_ext}link5">
+    <link name="link5">
       <visual>
         <origin xyz="0.0 0.0 0.0" rpy="0.0 0.0 0.0" />
@@ -205,7 +198,7 @@
       </inertial>
     </link>
-    <joint name="${tf_prefix_ext}gripper_left_joint" type="prismatic">
-      <parent link="${tf_prefix_ext}link5" />
-      <child link="${tf_prefix_ext}gripper_left_link" />
+    <joint name="gripper_left_joint" type="prismatic">
+      <parent link="link5" />
+      <child link="gripper_left_link" />
       <origin xyz="0.0817 0.021 0.0" rpy="0.0 0.0 0.0" />
       <axis xyz="0 1 0" />
@@ -213,5 +206,5 @@
       <dynamics damping="${damping}" />
     </joint>
-    <link name="${tf_prefix_ext}gripper_left_link">
+    <link name="gripper_left_link">
       <visual>
         <origin xyz="0.0 0.0 0.0" rpy="0.0 0.0 0.0" />
@@ -241,14 +234,14 @@
       </inertial>
     </link>
-    <joint name="${tf_prefix_ext}gripper_right_joint" type="prismatic">
-      <parent link="${tf_prefix_ext}link5" />
-      <child link="${tf_prefix_ext}gripper_right_link" />
+    <joint name="gripper_right_joint" type="prismatic">
+      <parent link="link5" />
+      <child link="gripper_right_link" />
       <origin xyz="0.0817 -0.021 0.0" rpy="0.0 0.0 0.0" />
       <axis xyz="0 -1 0" />
       <limit velocity="${velocity_limit}" effort="${effort_limit}" lower="-0.010" upper="0.019" />
-      <mimic joint="${tf_prefix_ext}gripper_left_joint" multiplier="1" />
-      <dynamics damping="${damping}" />
-    </joint>
-    <link name="${tf_prefix_ext}gripper_right_link">
+      <mimic joint="gripper_left_joint" multiplier="1" />
+      <dynamics damping="${damping}" />
+    </joint>
+    <link name="gripper_right_link">
       <visual>
         <origin xyz="0.0 0.0 0.0" rpy="0.0 0.0 0.0" />
@@ -278,14 +271,14 @@
       </inertial>
     </link>
-    <joint name="${tf_prefix_ext}end_effector_joint" type="fixed">
-      <parent link="${tf_prefix_ext}link5" />
-      <child link="${tf_prefix_ext}end_effector_link" />
+    <joint name="end_effector_joint" type="fixed">
+      <parent link="link5" />
+      <child link="end_effector_link" />
       <origin xyz="0.126 0.0 0.0" rpy="0.0 0.0 0.0" />
     </joint>
-    <link name="${tf_prefix_ext}end_effector_link" />
+    <link name="end_effector_link" />
     <ros2_control name="manipulator" type="system">
       <xacro:if value="$(arg use_sim)">
         <hardware>
-          <plugin>ign_ros2_control/IgnitionSystem</plugin>
+          <plugin>gz_ros2_control/GazeboSimSystem</plugin>
         </hardware>
       </xacro:if>
@@ -302,5 +295,5 @@
         </hardware>
       </xacro:unless>
-      <joint name="${tf_prefix_ext}joint1">
+      <joint name="joint1">
         <command_interface name="position">
           <param name="min">${joint1_limit_min}</param>
@@ -310,5 +303,5 @@
         <state_interface name="velocity" />
       </joint>
-      <joint name="${tf_prefix_ext}joint2">
+      <joint name="joint2">
         <command_interface name="position">
           <param name="min">${-pi*0.57}</param>
@@ -318,5 +311,5 @@
         <state_interface name="velocity" />
       </joint>
-      <joint name="${tf_prefix_ext}joint3">
+      <joint name="joint3">
         <command_interface name="position">
           <param name="min">${-pi*0.3}</param>
@@ -326,5 +319,5 @@
         <state_interface name="velocity" />
       </joint>
-      <joint name="${tf_prefix_ext}joint4">
+      <joint name="joint4">
         <command_interface name="position">
           <param name="min">${-pi*0.57}</param>
@@ -334,5 +327,5 @@
         <state_interface name="velocity" />
       </joint>
-      <joint name="${tf_prefix_ext}gripper_left_joint">
+      <joint name="gripper_left_joint">
         <command_interface name="position">
           <param name="min">-0.010</param>
