Commit message: Refactor open manipulator description

File: open_manipulator_x_description/urdf/open_manipulator_x.urdf.xacro (robot description, xacro)
@@ -1,8 +1,4 @@
 <?xml version="1.0"?>
-<!-- OpenManipulator-X -->
-<!--
-Copied and modified from open_manipulator-x example -
-https://github.com/ROBOTIS-GIT/open_manipulator/blob/kinetic-devel/open_manipulator_description/urdf/open_manipulator.urdf.xacro
--->
+<!-- based on https://github.com/ROBOTIS-GIT/open_manipulator -->
 <robot xmlns:xacro="http://www.ros.org/wiki/xacro">
   <xacro:macro name="open_manipulator_x"
@@ -16,4 +12,10 @@
       <xacro:property name="tf_prefix_ext" value="${tf_prefix}_" />
     </xacro:unless>
+    <material name="grey">
+      <color rgba="0.05 0.05 0.05 1.0" />
+    </material>
+    <xacro:property name="effort_limit" value="1" />
+    <xacro:property name="velocity_limit" value="4.8" />
+    <xacro:property name="damping" value="0.1" />
     <joint name="${parent_link}_to_${tf_prefix_ext}link1" type="fixed">
       <origin xyz="${xyz}" rpy="${rpy}" />
@@ -21,23 +23,17 @@
       <child link="${tf_prefix_ext}link1" />
     </joint>
-    <xacro:property
-      name="meshes_file_direction"
-      value="file://$(find open_manipulator_x_description)/meshes" />
-    <material name="grey">
-      <color rgba="0.05 0.05 0.05 1.0" />
-    </material>
     <link name="${tf_prefix_ext}link1">
       <visual>
         <origin xyz="0 0 0" rpy="0 0 0" />
         <geometry>
-          <mesh filename="${meshes_file_direction}/link1.stl" scale="0.001 0.001 0.001" />
-        </geometry>
-        <material name="grey" />
-      </visual>
-      <xacro:if value="${collision_enabled}">
-        <collision>
-          <origin xyz="0 0 0" rpy="0 0 0" />
-          <geometry>
-            <mesh filename="${meshes_file_direction}/link1.stl" scale="0.001 0.001 0.001" />
+          <mesh filename="file://$(find open_manipulator_x_description)/meshes/link1.stl" scale="0.001 0.001 0.001" />
+        </geometry>
+        <material name="grey" />
+      </visual>
+      <xacro:if value="${collision_enabled}">
+        <collision>
+          <origin xyz="0 0 0" rpy="0 0 0" />
+          <geometry>
+            <mesh filename="file://$(find open_manipulator_x_description)/meshes/link1.stl" scale="0.001 0.001 0.001" />
           </geometry>
         </collision>
@@ -56,6 +52,6 @@
       <origin xyz="0.012 0.0 0.017" rpy="0 0 0" />
       <axis xyz="0 0 1" />
-      <limit velocity="4.8" effort="1" lower="${-pi*205./180.}" upper="${pi*205./180.}" />
-      <dynamics damping="0.1" />
+      <limit velocity="${velocity_limit}" effort="${effort_limit}" lower="${-pi*205./180.}" upper="${pi*205./180.}" />
+      <dynamics damping="${damping}" />
     </joint>
     <link name="${tf_prefix_ext}link2">
@@ -63,5 +59,5 @@
         <origin xyz="0 0 0.019" rpy="0 0 0" />
         <geometry>
-          <mesh filename="${meshes_file_direction}/link2.stl" scale="0.001 0.001 0.001" />
+          <mesh filename="file://$(find open_manipulator_x_description)/meshes/link2.stl" scale="0.001 0.001 0.001" />
         </geometry>
         <material name="grey" />
@@ -72,5 +68,5 @@
           <geometry>
             <mesh
-              filename="${meshes_file_direction}/link2.stl" scale="0.001 0.001 0.001" />
+              filename="file://$(find open_manipulator_x_description)/meshes/link2.stl" scale="0.001 0.001 0.001" />
           </geometry>
         </collision>
@@ -89,6 +85,6 @@
       <origin xyz="0.0 0.0 0.0595" rpy="0 0 0" />
       <axis xyz="0 1 0" />
-      <limit velocity="4.8" effort="1" lower="${-pi*0.57}" upper="${pi*0.5}" />
-      <dynamics damping="0.1" />
+      <limit velocity="${velocity_limit}" effort="${effort_limit}" lower="${-pi*0.57}" upper="${pi*0.5}" />
+      <dynamics damping="${damping}" />
     </joint>
     <link name="${tf_prefix_ext}link3">
@@ -96,14 +92,14 @@
         <origin xyz="0 0 0" rpy="0 0 0" />
         <geometry>
-          <mesh filename="${meshes_file_direction}/link3.stl" scale="0.001 0.001 0.001" />
-        </geometry>
-        <material name="grey" />
-      </visual>
-      <xacro:if value="${collision_enabled}">
-        <collision>
-          <origin xyz="0 0 0" rpy="0 0 0" />
-          <geometry>
-            <mesh
-              filename="${meshes_file_direction}/link3.stl" scale="0.001 0.001 0.001" />
+          <mesh filename="file://$(find open_manipulator_x_description)/meshes/link3.stl" scale="0.001 0.001 0.001" />
+        </geometry>
+        <material name="grey" />
+      </visual>
+      <xacro:if value="${collision_enabled}">
+        <collision>
+          <origin xyz="0 0 0" rpy="0 0 0" />
+          <geometry>
+            <mesh
+              filename="file://$(find open_manipulator_x_description)/meshes/link3.stl" scale="0.001 0.001 0.001" />
           </geometry>
         </collision>
@@ -122,6 +118,6 @@
       <origin xyz="0.024 0 0.128" rpy="0 0 0" />
       <axis xyz="0 1 0" />
-      <limit velocity="4.8" effort="1" lower="${-pi*0.5}" upper="${pi*0.44}" />
-      <dynamics damping="0.1" />
+      <limit velocity="${velocity_limit}" effort="${effort_limit}" lower="${-pi*0.5}" upper="${pi*0.44}" />
+      <dynamics damping="${damping}" />
     </joint>
     <link name="${tf_prefix_ext}link4">
@@ -129,14 +125,14 @@
         <origin xyz="0 0 0" rpy="0 0 0" />
         <geometry>
-          <mesh filename="${meshes_file_direction}/link4.stl" scale="0.001 0.001 0.001" />
-        </geometry>
-        <material name="grey" />
-      </visual>
-      <xacro:if value="${collision_enabled}">
-        <collision>
-          <origin xyz="0 0 0" rpy="0 0 0" />
-          <geometry>
-            <mesh
-              filename="${meshes_file_direction}/link4.stl" scale="0.001 0.001 0.001" />
+          <mesh filename="file://$(find open_manipulator_x_description)/meshes/link4.stl" scale="0.001 0.001 0.001" />
+        </geometry>
+        <material name="grey" />
+      </visual>
+      <xacro:if value="${collision_enabled}">
+        <collision>
+          <origin xyz="0 0 0" rpy="0 0 0" />
+          <geometry>
+            <mesh
+              filename="file://$(find open_manipulator_x_description)/meshes/link4.stl" scale="0.001 0.001 0.001" />
           </geometry>
         </collision>
@@ -155,6 +151,6 @@
       <origin xyz="0.124 0.0 0.0" rpy="0 0 0" />
       <axis xyz="0 1 0" />
-      <limit velocity="4.8" effort="1" lower="${-pi*0.55}" upper="${pi*0.65}" />
-      <dynamics damping="0.1" />
+      <limit velocity="${velocity_limit}" effort="${effort_limit}" lower="${-pi*0.55}" upper="${pi*0.65}" />
+      <dynamics damping="${damping}" />
     </joint>
     <link name="${tf_prefix_ext}link5">
@@ -162,14 +158,14 @@
         <origin xyz="0 0 0" rpy="0 0 0" />
         <geometry>
-          <mesh filename="${meshes_file_direction}/link5.stl" scale="0.001 0.001 0.001" />
-        </geometry>
-        <material name="grey" />
-      </visual>
-      <xacro:if value="${collision_enabled}">
-        <collision>
-          <origin xyz="0 0 0" rpy="0 0 0" />
-          <geometry>
-            <mesh
-              filename="${meshes_file_direction}/link5.stl" scale="0.001 0.001 0.001" />
+          <mesh filename="file://$(find open_manipulator_x_description)/meshes/link5.stl" scale="0.001 0.001 0.001" />
+        </geometry>
+        <material name="grey" />
+      </visual>
+      <xacro:if value="${collision_enabled}">
+        <collision>
+          <origin xyz="0 0 0" rpy="0 0 0" />
+          <geometry>
+            <mesh
+              filename="file://$(find open_manipulator_x_description)/meshes/link5.stl" scale="0.001 0.001 0.001" />
           </geometry>
         </collision>
@@ -188,6 +184,6 @@
       <origin xyz="0.0817 0.021 0.0" rpy="0 0 0" />
       <axis xyz="0 1 0" />
-      <limit velocity="4.8" effort="1" lower="-0.010" upper="0.019" />
-      <dynamics damping="0.1" />
+      <limit velocity="${velocity_limit}" effort="${effort_limit}" lower="-0.010" upper="0.019" />
+      <dynamics damping="${damping}" />
     </joint>
     <link name="${tf_prefix_ext}gripper_left_link">
@@ -195,14 +191,14 @@
         <origin xyz="0 0 0" rpy="0 0 0" />
         <geometry>
-          <mesh filename="${meshes_file_direction}/gripper_left_palm.stl" scale="0.001 0.001 0.001" />
-        </geometry>
-        <material name="grey" />
-      </visual>
-      <xacro:if value="${collision_enabled}">
-        <collision>
-          <origin xyz="0 0 0" rpy="0 0 0" />
-          <geometry>
-            <mesh
-              filename="${meshes_file_direction}/gripper_left_palm.stl" scale="0.001 0.001 0.001" />
+          <mesh filename="file://$(find open_manipulator_x_description)/meshes/gripper_left_palm.stl" scale="0.001 0.001 0.001" />
+        </geometry>
+        <material name="grey" />
+      </visual>
+      <xacro:if value="${collision_enabled}">
+        <collision>
+          <origin xyz="0 0 0" rpy="0 0 0" />
+          <geometry>
+            <mesh
+              filename="file://$(find open_manipulator_x_description)/meshes/gripper_left_palm.stl" scale="0.001 0.001 0.001" />
           </geometry>
         </collision>
@@ -221,7 +217,7 @@
       <origin xyz="0.0817 -0.021 0" rpy="0 0 0" />
       <axis xyz="0 -1 0" />
-      <limit velocity="4.8" effort="1" lower="-0.010" upper="0.019" />
+      <limit velocity="${velocity_limit}" effort="${effort_limit}" lower="-0.010" upper="0.019" />
       <mimic joint="${tf_prefix_ext}gripper_left_joint" multiplier="1" />
-      <dynamics damping="0.1" />
+      <dynamics damping="${damping}" />
     </joint>
     <link name="${tf_prefix_ext}gripper_right_link">
@@ -229,14 +225,14 @@
         <origin xyz="0 0 0" rpy="0 0 0" />
         <geometry>
-          <mesh filename="${meshes_file_direction}/gripper_right_palm.stl" scale="0.001 0.001 0.001" />
-        </geometry>
-        <material name="grey" />
-      </visual>
-      <xacro:if value="${collision_enabled}">
-        <collision>
-          <origin xyz="0 0 0" rpy="0 0 0" />
-          <geometry>
-            <mesh
-              filename="${meshes_file_direction}/gripper_right_palm.stl" scale="0.001 0.001 0.001" />
+          <mesh filename="file://$(find open_manipulator_x_description)/meshes/gripper_right_palm.stl" scale="0.001 0.001 0.001" />
+        </geometry>
+        <material name="grey" />
+      </visual>
+      <xacro:if value="${collision_enabled}">
+        <collision>
+          <origin xyz="0 0 0" rpy="0 0 0" />
+          <geometry>
+            <mesh
+              filename="file://$(find open_manipulator_x_description)/meshes/gripper_right_palm.stl" scale="0.001 0.001 0.001" />
           </geometry>
         </collision>
@@ -255,14 +251,5 @@
       <origin xyz="0.126 0.0 0.0" rpy="0 0 0" />
     </joint>
-    <link name="${tf_prefix_ext}end_effector_link">
-      <!-- <visual>
-        <origin xyz="0 0 0" rpy="0 0 0" />
-        <geometry>
-          <box
-      size="0.01 0.01 0.01" />
-        </geometry>
-        <material name="red" />
-      </visual> -->
-    </link>
+    <link name="${tf_prefix_ext}end_effector_link" />
     <ros2_control name="manipulator" type="system">
       <xacro:if value="$(arg use_sim)">

Commit message: Remove second gripper joint from ros2 control
it only mimicked, isn't actuated

File: open_manipulator_x_description/urdf/open_manipulator_x.urdf.xacro (robot description, xacro)
@@ -310,14 +310,4 @@
         <state_interface name="velocity" />
       </joint>
-      <joint name="${tf_prefix_ext}gripper_right_joint">
-        <param name="mimic">gripper_left_joint</param>
-        <param name="multiplier">1</param>
-        <command_interface name="position">
-          <param name="min">-0.010</param>
-          <param name="max">0.019</param>
-        </command_interface>
-        <state_interface name="position" />
-        <state_interface name="velocity" />
-      </joint>
     </ros2_control>
   </xacro:macro>

Commit message: Simplify open_manipulator

File: open_manipulator_x_description/urdf/open_manipulator_x.urdf.xacro (robot description, xacro)
@@ -1,39 +1,231 @@
-<?xml version='1.0'?>
-<robot name="rosbot_xl" xmlns:xacro="http://www.ros.org/wiki/xacro">
-  <xacro:arg name="controller_config_file" default="$(find rosbot_xl_manipulation_controller)/config/diff_drive_controller_manipulation.yaml" />
-  <xacro:arg name="manipulator_usb_port" default="/dev/ttyUSB0" />
-  <xacro:arg name="manipulator_baud_rate" default="1000000" />
-  <!-- collision_enabled parameter added due to collisions using visual meshes, which are very
-    heavy and slow down simulation, this parameter allows to easily disable them -->
-  <xacro:arg name="manipulator_collision_enabled" default="true" />
-  <xacro:arg name="joint1_limit_min" default="-2.356" />
-  <xacro:arg name="joint1_limit_max" default="5.934" />
-  <xacro:arg name="use_sim" default="false" />
-  <xacro:arg name="namespace" default="" />
-  <link name="cover_link"/>
-  <xacro:include
-    filename="$(find open_manipulator_x_description)/urdf/open_manipulator_x_macro.urdf.xacro"
-    ns="manipulator" />
-  <xacro:manipulator.open_manipulator_x parent_link="cover_link"
-    xyz="-0.122 0.0 0.0"
-    rpy="0.0 0.0 0.0"
-    use_sim="$(arg use_sim)"
-    collision_enabled="$(arg manipulator_collision_enabled)"
-    usb_port="$(arg manipulator_usb_port)"
-    baud_rate="$(arg manipulator_baud_rate)"
-    joint1_limit_min="$(arg joint1_limit_min)"
-    joint1_limit_max="$(arg joint1_limit_max)" />
-  <xacro:if value="$(arg use_sim)">
-    <gazebo>
-      <plugin filename="gz_ros2_control-system" name="gz_ros2_control::GazeboSimROS2ControlPlugin">
-        <parameters>$(find open_manipulator_x_controller)/config/manipulator_controller.yaml</parameters>
-        <ros>
-          <namespace>$(arg namespace)</namespace>
-          <remapping>/diagnostics:=diagnostics</remapping>
-          <remapping>/tf:=tf</remapping>
-          <remapping>/tf_static:=tf_static</remapping>
-        </ros>
-      </plugin>
-    </gazebo>
-  </xacro:if>
+<?xml version="1.0"?>
+<robot xmlns:xacro="http://www.ros.org/wiki/xacro">
+  <xacro:macro name="open_manipulator_x" params="prefix='' parent_link=''">
+    <xacro:property
+      name="meshes_file_direction"
+      value="package://open_manipulator_x_description/meshes"/>
+    <xacro:if value="${parent_link != ''}">
+      <joint name="${prefix}${parent_link}" type="fixed">
+        <parent link="${parent_link}"/>
+        <child link="${prefix}link1"/>
+      </joint>
+    </xacro:if>
+    <link name="${prefix}link1">
+      <visual>
+        <origin xyz="0 0 0" rpy="0 0 0"/>
+        <geometry>
+          <mesh filename="${meshes_file_direction}/link1.stl" scale="0.001 0.001 0.001"/>
+        </geometry>
+        <material name="grey"/>
+      </visual>
+      <collision>
+        <origin xyz="0 0 0" rpy="0 0 0"/>
+        <geometry>
+          <mesh filename="${meshes_file_direction}/link1.stl" scale="0.001 0.001 0.001"/>
+        </geometry>
+      </collision>
+       <inertial>
+        <origin xyz="3.0876154e-04 0.0000000e+00 -1.2176461e-04" />
+        <mass value="7.9119962e-02" />
+        <inertia ixx="1.2505234e-05" ixy="0.0" ixz="-1.7855208e-07"
+                 iyy="2.1898364e-05" iyz="0.0"
+                 izz="1.9267361e-05" />
+      </inertial>
+    </link>
+    <joint name="${prefix}joint1" type="revolute">
+      <parent link="${prefix}link1"/>
+      <child link="${prefix}link2"/>
+      <origin xyz="0.012 0.0 0.017" rpy="0 0 0"/>
+      <axis xyz="0 0 1"/>
+      <limit velocity="4.8" effort="1" lower="${-pi}" upper="${pi}" />
+      <dynamics damping="0.1"/>
+    </joint>
+    <link name="${prefix}link2">
+      <visual>
+        <origin xyz="0 0 0.019" rpy="0 0 0"/>
+        <geometry>
+          <mesh filename="${meshes_file_direction}/link2.stl" scale="0.001 0.001 0.001"/>
+        </geometry>
+        <material name="grey"/>
+      </visual>
+      <collision>
+        <origin xyz="0 0 0.019" rpy="0 0 0"/>
+        <geometry>
+          <mesh filename="${meshes_file_direction}/link2.stl" scale="0.001 0.001 0.001"/>
+        </geometry>
+      </collision>
+       <inertial>
+        <origin xyz="-3.0184870e-04 5.4043684e-04 ${0.018 + 2.9433464e-02}" />
+        <mass value="9.8406837e-02" />
+        <inertia ixx="3.4543422e-05" ixy="-1.6031095e-08" ixz="-3.8375155e-07"
+                 iyy="3.2689329e-05" iyz="2.8511935e-08"
+                 izz="1.8850320e-05" />
+      </inertial>
+    </link>
+    <joint name="${prefix}joint2" type="revolute">
+      <parent link="${prefix}link2"/>
+      <child link="${prefix}link3"/>
+      <origin xyz="0.0 0.0 0.0595" rpy="0 0 0"/>
+      <axis xyz="0 1 0"/>
+      <limit velocity="4.8" effort="1" lower="${-1.5}" upper="${1.5}" />
+      <dynamics damping="0.1"/>
+    </joint>
+    <link name="${prefix}link3">
+      <visual>
+        <origin xyz="0 0 0" rpy="0 0 0"/>
+        <geometry>
+          <mesh filename="${meshes_file_direction}/link3.stl" scale="0.001 0.001 0.001"/>
+        </geometry>
+        <material name="grey"/>
+      </visual>
+      <collision>
+        <origin xyz="0 0 0" rpy="0 0 0"/>
+        <geometry>
+          <mesh filename="${meshes_file_direction}/link3.stl" scale="0.001 0.001 0.001"/>
+        </geometry>
+      </collision>
+       <inertial>
+        <origin xyz="1.0308393e-02 3.7743363e-04 1.0170197e-01" />
+        <mass value="1.3850917e-01" />
+        <inertia ixx="3.3055381e-04" ixy="-9.7940978e-08" ixz="-3.8505711e-05"
+                 iyy="3.4290447e-04" iyz="-1.5717516e-06"
+                 izz="6.0346498e-05" />
+      </inertial>
+    </link>
+    <joint name="${prefix}joint3" type="revolute">
+      <parent link="${prefix}link3"/>
+      <child link="${prefix}link4"/>
+      <origin xyz="0.024 0 0.128" rpy="0 0 0"/>
+      <axis xyz="0 1 0"/>
+      <limit velocity="4.8" effort="1" lower="${-1.5}" upper="${1.4}" />
+      <dynamics damping="0.1"/>
+    </joint>
+    <link name="${prefix}link4">
+      <visual>
+        <origin xyz="0 0 0" rpy="0 0 0"/>
+        <geometry>
+          <mesh filename="${meshes_file_direction}/link4.stl" scale="0.001 0.001 0.001"/>
+        </geometry>
+        <material name="grey"/>
+      </visual>
+      <collision>
+        <origin xyz="0 0 0" rpy="0 0 0"/>
+        <geometry>
+          <mesh filename="${meshes_file_direction}/link4.stl" scale="0.001 0.001 0.001"/>
+        </geometry>
+      </collision>
+       <inertial>
+        <origin xyz="9.0909590e-02 3.8929816e-04 2.2413279e-04" />
+        <mass value="1.3274562e-01" />
+        <inertia ixx="3.0654178e-05" ixy="-1.2764155e-06" ixz="-2.6874417e-07"
+                 iyy="2.4230292e-04" iyz="1.1559550e-08"
+                 izz="2.5155057e-04" />
+      </inertial>
+    </link>
+    <joint name="${prefix}joint4" type="revolute">
+      <parent link="${prefix}link4"/>
+      <child link="${prefix}link5"/>
+      <origin xyz="0.124 0.0 0.0" rpy="0 0 0"/>
+      <axis xyz="0 1 0"/>
+      <limit velocity="4.8" effort="1" lower="${-1.7}" upper="${1.97}" />
+      <dynamics damping="0.1"/>
+    </joint>
+    <link name="${prefix}link5">
+      <visual>
+        <origin xyz="0 0 0" rpy="0 0 0"/>
+        <geometry>
+          <mesh filename="${meshes_file_direction}/link5.stl" scale="0.001 0.001 0.001"/>
+        </geometry>
+        <material name="grey"/>
+      </visual>
+      <collision>
+        <origin xyz="0 0 0" rpy="0 0 0"/>
+        <geometry>
+          <mesh filename="${meshes_file_direction}/link5.stl" scale="0.001 0.001 0.001"/>
+        </geometry>
+      </collision>
+       <inertial>
+        <origin xyz="4.4206755e-02 3.6839985e-07 8.9142216e-03" />
+        <mass value="1.4327573e-01" />
+        <inertia ixx="8.0870749e-05" ixy="0.0" ixz="-1.0157896e-06"
+                 iyy="7.5980465e-05" iyz="0.0"
+                 izz="9.3127351e-05" />
+      </inertial>
+    </link>
+    <joint name="${prefix}gripper_left_joint" type="prismatic">
+      <parent link="${prefix}link5"/>
+      <child link="${prefix}gripper_left_link"/>
+      <origin xyz="0.0817 0.021 0.0" rpy="0 0 0"/>
+      <axis xyz="0 1 0"/>
+      <limit velocity="4.8" effort="1" lower="-0.010" upper="0.019" />
+      <dynamics damping="0.1"/>
+    </joint>
+    <link name="${prefix}gripper_left_link">
+      <visual>
+        <origin xyz="0 0 0" rpy="0 0 0"/>
+        <geometry>
+          <mesh filename="${meshes_file_direction}/gripper_left_palm.stl" scale="0.001 0.001 0.001"/>
+        </geometry>
+        <material name="grey"/>
+      </visual>
+      <collision>
+        <origin xyz="0 0 0" rpy="0 0 0"/>
+        <geometry>
+          <mesh filename="${meshes_file_direction}/gripper_left_palm.stl" scale="0.001 0.001 0.001"/>
+        </geometry>
+      </collision>
+      <inertial>
+        <origin xyz="0 0 0" />
+        <mass value="1.0e-03" />
+        <inertia ixx="1.0e-06" ixy="0.0" ixz="0.0"
+                 iyy="1.0e-06" iyz="0.0"
+                 izz="1.0e-06" />
+      </inertial>
+    </link>
+    <joint name="${prefix}gripper_right_joint" type="prismatic">
+      <parent link="${prefix}link5"/>
+      <child link="${prefix}gripper_right_link"/>
+      <origin xyz="0.0817 -0.021 0" rpy="0 0 0"/>
+      <axis xyz="0 -1 0"/>
+      <limit velocity="4.8" effort="1" lower="-0.010" upper="0.019" />
+      <!-- <mimic joint="${prefix}gripper_left_joint" multiplier="1"/> -->
+      <dynamics damping="0.1"/>
+    </joint>
+    <link name="${prefix}gripper_right_link">
+      <visual>
+        <origin xyz="0 0 0" rpy="0 0 0"/>
+        <geometry>
+          <mesh filename="${meshes_file_direction}/gripper_right_palm.stl" scale="0.001 0.001 0.001"/>
+        </geometry>
+        <material name="grey"/>
+      </visual>
+      <collision>
+        <origin xyz="0 0 0" rpy="0 0 0"/>
+        <geometry>
+          <mesh filename="${meshes_file_direction}/gripper_right_palm.stl" scale="0.001 0.001 0.001"/>
+        </geometry>
+      </collision>
+      <inertial>
+        <origin xyz="0 0 0" />
+        <mass value="1.0e-03" />
+        <inertia ixx="1.0e-06" ixy="0.0" ixz="0.0"
+                 iyy="1.0e-06" iyz="0.0"
+                 izz="1.0e-06" />
+      </inertial>
+    </link>
+    <joint name="${prefix}end_effector_joint" type="fixed">
+      <parent link="${prefix}link5"/>
+      <child link="${prefix}end_effector_link"/>
+      <origin xyz="0.126 0.0 0.0" rpy="0 0 0"/>
+    </joint>
+    <link name="${prefix}end_effector_link">
+      <visual>
+        <origin xyz="0 0 0" rpy="0 0 0"/>
+        <geometry>
+          <box size="0.01 0.01 0.01" />
+        </geometry>
+        <material name="red"/>
+       </visual>
+    </link>
+  </xacro:macro>
 </robot>
