Commit message: Save work

File: open_manipulator_x_description/urdf/ros2_control.xacro (robot description, xacro)
@@ -22,5 +22,5 @@
             <param name="error_timeout_ms">500</param>
             <param name="dynamixel_model_folder">/param/dxl_model</param>
-            <param name="number_of_joints">5</param>
+            <param name="number_of_joints">6</param>
             <param name="number_of_transmissions">5</param>
             <param name="transmission_to_joint_matrix">
@@ -29,12 +29,13 @@
               0, 0, 1, 0, 0,
               0, 0, 0, 1, 0,
-              0, 0, 0, 0, 1
+              0, 0, 0, 0, 1,
+              0, 0, 0, 0, 0
             </param>
             <param name="joint_to_transmission_matrix">
-              1, 0, 0, 0, 0,
-              0, 1, 0, 0, 0,
-              0, 0, 1, 0, 0,
-              0, 0, 0, 1, 0,
-              0, 0, 0, 0, 1
+              1, 0, 0, 0, 0, 0,
+              0, 1, 0, 0, 0, 0,
+              0, 0, 1, 0, 0, 0,
+              0, 0, 0, 1, 0, 0,
+              0, 0, 0, 0, 1, 0
             </param>
             <param name="ros_update_freq">200</param>
@@ -86,4 +87,12 @@
         <state_interface name="effort"/>
       </joint>
+      <joint name="${prefix}gripper_right_joint">
+        <param name="mimic">${prefix}gripper_left_joint</param>
+        <param name="multiplier">1</param>
+        <command_interface name="position"/>
+        <state_interface name="position"/>
+        <state_interface name="velocity"/>
+        <state_interface name="effort"/>
+      </joint>
       <gpio name="dxl1">
         <param name="type">dxl</param>
@@ -101,4 +110,5 @@
         <param name="Profile Acceleration">50</param>
         <param name="Drive Mode">0</param>
+        <param name="Return Delay Time">0</param>
       </gpio>
       <gpio name="dxl2">
@@ -117,4 +127,5 @@
         <param name="Profile Acceleration">50</param>
         <param name="Drive Mode">0</param>
+        <param name="Return Delay Time">0</param>
       </gpio>
       <gpio name="dxl3">
@@ -133,4 +144,5 @@
         <param name="Profile Acceleration">50</param>
         <param name="Drive Mode">0</param>
+        <param name="Return Delay Time">0</param>
       </gpio>
       <gpio name="dxl4">
@@ -149,4 +161,5 @@
         <param name="Profile Acceleration">50</param>
         <param name="Drive Mode">0</param>
+        <param name="Return Delay Time">0</param>
       </gpio>
       <gpio name="dxl5">
@@ -159,4 +172,5 @@
         <state_interface name="Torque Enable"/>
         <state_interface name="Present Input Voltage"/>
+        <param name="Return Delay Time">0</param>
       </gpio>
     </ros2_control>

Commit message: Great update Open Manipulation for ROSbot XL Manipulation

File: open_manipulator_x_description/urdf/ros2_control.xacro (robot description, xacro)
@@ -38,5 +38,4 @@
               0, 0, 0, 0, 1
             </param>
-            <param name="ros_update_freq">200</param>
             <param name="dynamixel_state_pub_msg_name">dynamixel_hardware_interface/dxl_state</param>
             <param name="get_dynamixel_data_srv_name">dynamixel_hardware_interface/get_dxl_data</param>
@@ -44,6 +43,6 @@
             <param name="reboot_dxl_srv_name">dynamixel_hardware_interface/reboot_dxl</param>
             <param name="set_dxl_torque_srv_name">dynamixel_hardware_interface/set_dxl_torque</param>
-              <!-- This parameter is used for a prismatic joint
-            that operates through a revolute mechanism. If the joint does not require this configuration, this parameter can be removed. -->
+            <!-- This parameter is used for a prismatic joint that operates through a revolute mechanism.
+            If the joint does not require this configuration, this parameter can be removed. -->
             <param name="use_revolute_to_prismatic_gripper">1</param>
             <param name="revolute_to_prismatic_dxl">dxl5</param>
@@ -86,4 +85,13 @@
         <state_interface name="effort"/>
       </joint>
+      <xacro:if value="$(arg use_sim)">
+        <joint name="${prefix}gripper_right_joint">
+          <param name="mimic">${prefix}gripper_left_joint</param>
+          <param name="multiplier">1</param>
+          <state_interface name="position"/>
+          <state_interface name="velocity"/>
+          <state_interface name="effort"/>
+        </joint>
+      </xacro:if>
       <gpio name="dxl1">
         <param name="type">dxl</param>

Commit message: Remove gripper_right_joint

File: open_manipulator_x_description/urdf/ros2_control.xacro (robot description, xacro)
@@ -22,5 +22,5 @@
             <param name="error_timeout_ms">5000</param>
             <param name="dynamixel_model_folder">/param/dxl_model</param>
-            <param name="number_of_joints">6</param>
+            <param name="number_of_joints">5</param>
             <param name="number_of_transmissions">5</param>
             <param name="transmission_to_joint_matrix">
@@ -29,13 +29,12 @@
               0, 0, 1, 0, 0,
               0, 0, 0, 1, 0,
-              0, 0, 0, 0, 1,
-              0, 0, 0, 0, 0
+              0, 0, 0, 0, 1
             </param>
             <param name="joint_to_transmission_matrix">
-              1, 0, 0, 0, 0, 0,
-              0, 1, 0, 0, 0, 0,
-              0, 0, 1, 0, 0, 0,
-              0, 0, 0, 1, 0, 0,
-              0, 0, 0, 0, 1, 0
+              1, 0, 0, 0, 0,
+              0, 1, 0, 0, 0,
+              0, 0, 1, 0, 0,
+              0, 0, 0, 1, 0,
+              0, 0, 0, 0, 1
             </param>
             <param name="ros_update_freq">200</param>
@@ -82,10 +81,4 @@
       </joint>
       <joint name="${prefix}gripper_left_joint">
-        <command_interface name="position"/>
-        <state_interface name="position"/>
-        <state_interface name="velocity"/>
-        <state_interface name="effort"/>
-      </joint>
-      <joint name="${prefix}gripper_right_joint">
         <command_interface name="position"/>
         <state_interface name="position"/>
