Commit message: Refactor

File: open_manipulator_x_description/urdf/body.xacro (robot description, xacro)
@@ -1,10 +1,14 @@
 <?xml version="1.0"?>
 <robot xmlns:xacro="http://www.ros.org/wiki/xacro">
-  <xacro:macro name="open_manipulator_x" params="prefix='' parent_link=''">
-    <xacro:property
-      name="meshes_file_direction"
-      value="package://open_manipulator_x_description/meshes"/>
+  <xacro:macro name="open_manipulator_x"
+            params="parent_link=''
+                    xyz:='0.0 0.0 0.0'
+                    rpy:='0.0 0.0 0.0'
+                    namespace:=''
+                    prefix:=''">
+    <xacro:property name="meshes_dir" value="package://open_manipulator_x_description/meshes"/>
     <xacro:if value="${parent_link != ''}">
       <joint name="${prefix}${parent_link}" type="fixed">
+        <origin xyz="${xyz}" rpy="${rpy}" />
         <parent link="${parent_link}"/>
         <child link="${prefix}link1"/>
@@ -15,12 +19,12 @@
         <origin xyz="0 0 0" rpy="0 0 0"/>
         <geometry>
-          <mesh filename="${meshes_file_direction}/link1.stl" scale="0.001 0.001 0.001"/>
-        </geometry>
-        <material name="grey"/>
-      </visual>
-      <collision>
-        <origin xyz="0 0 0" rpy="0 0 0"/>
-        <geometry>
-          <mesh filename="${meshes_file_direction}/link1.stl" scale="0.001 0.001 0.001"/>
+          <mesh filename="${meshes_dir}/link1.stl" scale="0.001 0.001 0.001"/>
+        </geometry>
+        <material name="grey"/>
+      </visual>
+      <collision>
+        <origin xyz="0 0 0" rpy="0 0 0"/>
+        <geometry>
+          <mesh filename="${meshes_dir}/link1.stl" scale="0.001 0.001 0.001"/>
         </geometry>
       </collision>
@@ -45,5 +49,5 @@
         <origin xyz="0 0 0.019" rpy="0 0 0"/>
         <geometry>
-          <mesh filename="${meshes_file_direction}/link2.stl" scale="0.001 0.001 0.001"/>
+          <mesh filename="${meshes_dir}/link2.stl" scale="0.001 0.001 0.001"/>
         </geometry>
         <material name="grey"/>
@@ -52,5 +56,5 @@
         <origin xyz="0 0 0.019" rpy="0 0 0"/>
         <geometry>
-          <mesh filename="${meshes_file_direction}/link2.stl" scale="0.001 0.001 0.001"/>
+          <mesh filename="${meshes_dir}/link2.stl" scale="0.001 0.001 0.001"/>
         </geometry>
       </collision>
@@ -75,12 +79,12 @@
         <origin xyz="0 0 0" rpy="0 0 0"/>
         <geometry>
-          <mesh filename="${meshes_file_direction}/link3.stl" scale="0.001 0.001 0.001"/>
-        </geometry>
-        <material name="grey"/>
-      </visual>
-      <collision>
-        <origin xyz="0 0 0" rpy="0 0 0"/>
-        <geometry>
-          <mesh filename="${meshes_file_direction}/link3.stl" scale="0.001 0.001 0.001"/>
+          <mesh filename="${meshes_dir}/link3.stl" scale="0.001 0.001 0.001"/>
+        </geometry>
+        <material name="grey"/>
+      </visual>
+      <collision>
+        <origin xyz="0 0 0" rpy="0 0 0"/>
+        <geometry>
+          <mesh filename="${meshes_dir}/link3.stl" scale="0.001 0.001 0.001"/>
         </geometry>
       </collision>
@@ -105,12 +109,12 @@
         <origin xyz="0 0 0" rpy="0 0 0"/>
         <geometry>
-          <mesh filename="${meshes_file_direction}/link4.stl" scale="0.001 0.001 0.001"/>
-        </geometry>
-        <material name="grey"/>
-      </visual>
-      <collision>
-        <origin xyz="0 0 0" rpy="0 0 0"/>
-        <geometry>
-          <mesh filename="${meshes_file_direction}/link4.stl" scale="0.001 0.001 0.001"/>
+          <mesh filename="${meshes_dir}/link4.stl" scale="0.001 0.001 0.001"/>
+        </geometry>
+        <material name="grey"/>
+      </visual>
+      <collision>
+        <origin xyz="0 0 0" rpy="0 0 0"/>
+        <geometry>
+          <mesh filename="${meshes_dir}/link4.stl" scale="0.001 0.001 0.001"/>
         </geometry>
       </collision>
@@ -135,12 +139,12 @@
         <origin xyz="0 0 0" rpy="0 0 0"/>
         <geometry>
-          <mesh filename="${meshes_file_direction}/link5.stl" scale="0.001 0.001 0.001"/>
-        </geometry>
-        <material name="grey"/>
-      </visual>
-      <collision>
-        <origin xyz="0 0 0" rpy="0 0 0"/>
-        <geometry>
-          <mesh filename="${meshes_file_direction}/link5.stl" scale="0.001 0.001 0.001"/>
+          <mesh filename="${meshes_dir}/link5.stl" scale="0.001 0.001 0.001"/>
+        </geometry>
+        <material name="grey"/>
+      </visual>
+      <collision>
+        <origin xyz="0 0 0" rpy="0 0 0"/>
+        <geometry>
+          <mesh filename="${meshes_dir}/link5.stl" scale="0.001 0.001 0.001"/>
         </geometry>
       </collision>
@@ -165,12 +169,12 @@
         <origin xyz="0 0 0" rpy="0 0 0"/>
         <geometry>
-          <mesh filename="${meshes_file_direction}/gripper_left_palm.stl" scale="0.001 0.001 0.001"/>
-        </geometry>
-        <material name="grey"/>
-      </visual>
-      <collision>
-        <origin xyz="0 0 0" rpy="0 0 0"/>
-        <geometry>
-          <mesh filename="${meshes_file_direction}/gripper_left_palm.stl" scale="0.001 0.001 0.001"/>
+          <mesh filename="${meshes_dir}/gripper_left_palm.stl" scale="0.001 0.001 0.001"/>
+        </geometry>
+        <material name="grey"/>
+      </visual>
+      <collision>
+        <origin xyz="0 0 0" rpy="0 0 0"/>
+        <geometry>
+          <mesh filename="${meshes_dir}/gripper_left_palm.stl" scale="0.001 0.001 0.001"/>
         </geometry>
       </collision>
@@ -196,12 +200,12 @@
         <origin xyz="0 0 0" rpy="0 0 0"/>
         <geometry>
-          <mesh filename="${meshes_file_direction}/gripper_right_palm.stl" scale="0.001 0.001 0.001"/>
-        </geometry>
-        <material name="grey"/>
-      </visual>
-      <collision>
-        <origin xyz="0 0 0" rpy="0 0 0"/>
-        <geometry>
-          <mesh filename="${meshes_file_direction}/gripper_right_palm.stl" scale="0.001 0.001 0.001"/>
+          <mesh filename="${meshes_dir}/gripper_right_palm.stl" scale="0.001 0.001 0.001"/>
+        </geometry>
+        <material name="grey"/>
+      </visual>
+      <collision>
+        <origin xyz="0 0 0" rpy="0 0 0"/>
+        <geometry>
+          <mesh filename="${meshes_dir}/gripper_right_palm.stl" scale="0.001 0.001 0.001"/>
         </geometry>
       </collision>

File: open_manipulator_x_description/urdf/gazebo.xacro (robot description, xacro)
@@ -5,5 +5,5 @@
 -->
 <robot xmlns:xacro="http://ros.org/wiki/xacro">
-  <xacro:macro name="open_manipulator_x_gazebo" params="prefix">
+  <xacro:macro name="gz_open_manipulator_x_system" params="prefix:=''">
   <xacro:macro name="SimpleTransmission" params="trans joint actuator">
     <transmission name="${trans}">

File: open_manipulator_x_description/urdf/open_manipulator_x_robot.urdf.xacro (robot description, xacro)
@@ -7,15 +7,8 @@
   <xacro:arg name="fake_sensor_commands" default="false" />
   <xacro:arg name="port_name" default="/dev/ttyUSB0" />
-  <!-- Import Rviz colors -->
-  <xacro:include filename="$(find open_manipulator_x_description)/urdf/materials.xacro" />
-  <!-- Import all Gazebo-customization elements, including Gazebo colors -->
-  <xacro:include filename="$(find open_manipulator_x_description)/urdf/open_manipulator_x.gazebo.xacro" />
-  <!-- Import URDF -->
-  <xacro:include filename="$(find open_manipulator_x_description)/urdf/open_manipulator_x.urdf.xacro" />
-  <xacro:include filename="$(find open_manipulator_x_description)/urdf/open_manipulator_x_system.ros2_control.xacro" />
-  <xacro:open_manipulator_x prefix="$(arg prefix)" />
-  <xacro:open_manipulator_x_gazebo prefix="$(arg prefix)" />
-  <xacro:open_manipulator_x_system
-    name="OpenManipulatorXSystem" prefix="$(arg prefix)" use_sim="$(arg use_sim)"
+  <xacro:include filename="$(find open_manipulator_x_description)/urdf/open_manipulator_x_macro.xacro" />
+  <xacro:open_manipulator_x
+    device_namespace="$(arg prefix)"
+    use_sim="$(arg use_sim)"
     use_fake_hardware="$(arg use_fake_hardware)"
     fake_sensor_commands="$(arg fake_sensor_commands)"

File: open_manipulator_x_description/urdf/ros2_control.xacro (robot description, xacro)
@@ -1,6 +1,7 @@
 <?xml version="1.0"?>
 <robot xmlns:xacro="http://www.ros.org/wiki/xacro">
-  <xacro:macro name="open_manipulator_x_system" params="name prefix port_name:=/dev/ttyUSB0 use_sim:=^|false use_fake_hardware:=^|false fake_sensor_commands:=^|false">
-    <ros2_control name="${name}" type="system">
+  <xacro:macro name="open_manipulator_x_system" params="name:='OpenManipulatorXSystem' namespace:='' prefix:='' port_name:=/dev/ttyUSB0 use_sim:=^|false use_fake_hardware:=^|false fake_sensor_commands:=^|false">
+    <xacro:property name="ns" value="${namespace + '/' if namespace != '' else ''}" />
+    <ros2_control name="${ns}${name}" type="system">
       <xacro:if value="$(arg use_sim)">
         <hardware>
@@ -19,5 +20,5 @@
             <param name="port_name">${port_name}</param>
             <param name="baud_rate">1000000</param>
-            <param name="error_timeout_sec">0.2</param>
+            <param name="error_timeout_ms">500</param>
             <param name="dynamixel_model_folder">/param/dxl_model</param>
             <param name="number_of_joints">6</param>

Commit message: Add custom cylinder base and fix origin

File: open_manipulator_x_description/urdf/body.xacro (robot description, xacro)
@@ -17,14 +17,18 @@
     <link name="${prefix}link1">
       <visual>
-        <origin xyz="0 0 0" rpy="0 0 0"/>
-        <geometry>
-          <mesh filename="${meshes_dir}/link1.stl" scale="0.001 0.001 0.001"/>
-        </geometry>
-        <material name="grey"/>
-      </visual>
-      <collision>
-        <origin xyz="0 0 0" rpy="0 0 0"/>
-        <geometry>
-          <mesh filename="${meshes_dir}/link1.stl" scale="0.001 0.001 0.001"/>
+        <origin xyz="0 0 0.03" rpy="0 0 0"/>
+        <geometry>
+          <!-- We use custom cylinder -->
+          <cylinder radius="0.035" length="0.065" />
+          <!-- <mesh filename="${meshes_dir}/link1.stl" scale="0.001 0.001 0.001"/> -->
+        </geometry>
+        <material name="grey"/>
+      </visual>
+      <collision>
+        <origin xyz="0 0 0.03" rpy="0 0 0"/>
+        <geometry>
+          <!-- We use custom cylinder -->
+          <cylinder radius="0.035" length="0.065" />
+          <!-- <mesh filename="${meshes_dir}/link1.stl" scale="0.001 0.001 0.001"/> -->
         </geometry>
       </collision>
@@ -40,5 +44,6 @@
       <parent link="${prefix}link1"/>
       <child link="${prefix}link2"/>
-      <origin xyz="0.012 0.0 0.017" rpy="0 0 0"/>
+      <!-- Fix origin on custom cylinder -->
+      <origin xyz="0.0 0.0 0.045" rpy="0 0 0"/>
       <axis xyz="0 0 1"/>
       <limit velocity="4.8" effort="1" lower="${-pi}" upper="${pi}" />
@@ -47,5 +52,5 @@
     <link name="${prefix}link2">
       <visual>
-        <origin xyz="0 0 0.019" rpy="0 0 0"/>
+        <origin xyz="0 0 0" rpy="0 0 0"/>
         <geometry>
           <mesh filename="${meshes_dir}/link2.stl" scale="0.001 0.001 0.001"/>
@@ -54,5 +59,5 @@
       </visual>
       <collision>
-        <origin xyz="0 0 0.019" rpy="0 0 0"/>
+        <origin xyz="0 0 0" rpy="0 0 0"/>
         <geometry>
           <mesh filename="${meshes_dir}/link2.stl" scale="0.001 0.001 0.001"/>

Commit message: Fix right gripper mimic left griper

File: open_manipulator_x_description/urdf/body.xacro (robot description, xacro)
@@ -198,5 +198,5 @@
       <axis xyz="0 -1 0"/>
       <limit velocity="4.8" effort="1" lower="-0.010" upper="0.019" />
-      <!-- <mimic joint="${prefix}gripper_left_joint" multiplier="1"/> -->
+      <mimic joint="${prefix}gripper_left_joint" multiplier="1"/>
       <dynamics damping="0.1"/>
     </joint>

File: open_manipulator_x_description/urdf/ros2_control.xacro (robot description, xacro)
@@ -22,5 +22,5 @@
             <param name="error_timeout_ms">500</param>
             <param name="dynamixel_model_folder">/param/dxl_model</param>
-            <param name="number_of_joints">6</param>
+            <param name="number_of_joints">5</param>
             <param name="number_of_transmissions">5</param>
             <param name="transmission_to_joint_matrix">
@@ -29,13 +29,12 @@
               0, 0, 1, 0, 0,
               0, 0, 0, 1, 0,
-              0, 0, 0, 0, 1,
-              0, 0, 0, 0, 0
+              0, 0, 0, 0, 1
             </param>
             <param name="joint_to_transmission_matrix">
-              1, 0, 0, 0, 0, 0,
-              0, 1, 0, 0, 0, 0,
-              0, 0, 1, 0, 0, 0,
-              0, 0, 0, 1, 0, 0,
-              0, 0, 0, 0, 1, 0
+              1, 0, 0, 0, 0,
+              0, 1, 0, 0, 0,
+              0, 0, 1, 0, 0,
+              0, 0, 0, 1, 0,
+              0, 0, 0, 0, 1
             </param>
             <param name="ros_update_freq">200</param>
@@ -87,10 +86,4 @@
         <state_interface name="effort"/>
       </joint>
-      <joint name="${prefix}gripper_right_joint">
-        <command_interface name="position"/>
-        <state_interface name="position"/>
-        <state_interface name="velocity"/>
-        <state_interface name="effort"/>
-      </joint>
       <gpio name="dxl1">
         <param name="type">dxl</param>
@@ -105,4 +98,6 @@
         <param name="Position I Gain">100</param>
         <param name="Position D Gain">100</param>
+        <param name="Profile Velocity">200</param>
+        <param name="Profile Acceleration">50</param>
         <param name="Drive Mode">0</param>
       </gpio>
@@ -119,4 +114,6 @@
         <param name="Position I Gain">100</param>
         <param name="Position D Gain">100</param>
+        <param name="Profile Velocity">200</param>
+        <param name="Profile Acceleration">50</param>
         <param name="Drive Mode">0</param>
       </gpio>
@@ -133,4 +130,6 @@
         <param name="Position I Gain">100</param>
         <param name="Position D Gain">100</param>
+        <param name="Profile Velocity">200</param>
+        <param name="Profile Acceleration">50</param>
         <param name="Drive Mode">0</param>
       </gpio>
@@ -147,4 +146,6 @@
         <param name="Position I Gain">100</param>
         <param name="Position D Gain">100</param>
+        <param name="Profile Velocity">200</param>
+        <param name="Profile Acceleration">50</param>
         <param name="Drive Mode">0</param>
       </gpio>

Commit message: Simulation fixes

File: open_manipulator_x_description/urdf/body.xacro (robot description, xacro)
@@ -9,5 +9,5 @@
     <xacro:property name="meshes_dir" value="package://open_manipulator_x_description/meshes"/>
     <xacro:if value="${parent_link != ''}">
-      <joint name="${prefix}${parent_link}" type="fixed">
+      <joint name="${prefix}${parent_link}_joint" type="fixed">
         <origin xyz="${xyz}" rpy="${rpy}" />
         <parent link="${parent_link}"/>
@@ -235,5 +235,5 @@
         </geometry>
         <material name="red"/>
-       </visual>
+      </visual>
     </link>
   </xacro:macro>

File: open_manipulator_x_description/urdf/open_manipulator_x_macro.xacro (robot description, xacro)
@@ -25,13 +25,11 @@
       rpy="${rpy}" />
     <!-- ROS2 CONTROL PLUGINS -->
-    <xacro:unless value="${use_sim}">
-      <xacro:ros2_control.open_manipulator_x_system
-        name="OpenManipulatorXSystem"
-        prefix="${prefix}"
-        use_sim="${use_sim}"
-        use_fake_hardware="${use_fake_hardware}"
-        fake_sensor_commands="${fake_sensor_commands}"
-        port_name="${port_name}" />
-    </xacro:unless>
+    <xacro:ros2_control.open_manipulator_x_system
+      name="OpenManipulatorXSystem"
+      prefix="${prefix}"
+      use_sim="${use_sim}"
+      use_fake_hardware="${use_fake_hardware}"
+      fake_sensor_commands="${fake_sensor_commands}"
+      port_name="${port_name}" />
     <!-- GAZEBO PLUGINS -->
     <xacro:if value="${use_sim}">

File: open_manipulator_x_description/urdf/ros2_control.xacro (robot description, xacro)
@@ -6,5 +6,5 @@
       <xacro:if value="$(arg use_sim)">
         <hardware>
-          <plugin>gazebo_ros2_control/GazeboSystem</plugin>
+          <plugin>gz_ros2_control/GazeboSimSystem</plugin>
         </hardware>
       </xacro:if>

Commit message: Remove end_of_effector visualization

File: open_manipulator_x_description/urdf/body.xacro (robot description, xacro)
@@ -228,13 +228,5 @@
       <origin xyz="0.126 0.0 0.0" rpy="0 0 0"/>
     </joint>
-    <link name="${prefix}end_effector_link">
-      <visual>
-        <origin xyz="0 0 0" rpy="0 0 0"/>
-        <geometry>
-          <box size="0.01 0.01 0.01" />
-        </geometry>
-        <material name="red"/>
-      </visual>
-    </link>
+    <link name="${prefix}end_effector_link"/>
   </xacro:macro>
 </robot>

Commit message: Manipulator working fine

File: open_manipulator_x_description/urdf/body.xacro (robot description, xacro)
@@ -9,5 +9,5 @@
     <xacro:property name="meshes_dir" value="package://open_manipulator_x_description/meshes"/>
     <xacro:if value="${parent_link != ''}">
-      <joint name="${prefix}${parent_link}_joint" type="fixed">
+      <joint name="${prefix}${parent_link}_to_link1" type="fixed">
         <origin xyz="${xyz}" rpy="${rpy}" />
         <parent link="${parent_link}"/>

File: open_manipulator_x_description/urdf/ros2_control.xacro (robot description, xacro)
@@ -6,5 +6,5 @@
       <xacro:if value="$(arg use_sim)">
         <hardware>
-          <plugin>ign_ros2_control/IgnitionSystem</plugin>
+          <plugin>gz_ros2_control/GazeboSimSystem</plugin>
         </hardware>
       </xacro:if>
@@ -88,6 +88,4 @@
       </joint>
       <joint name="${prefix}gripper_right_joint">
-        <param name="mimic">${prefix}gripper_left_joint</param>
-        <param name="multiplier">1</param>
         <command_interface name="position"/>
         <state_interface name="position"/>

Commit message: Improve URDF

File: open_manipulator_x_description/urdf/body.xacro (robot description, xacro)
@@ -8,4 +8,5 @@
                     prefix:=''">
     <xacro:property name="meshes_dir" value="package://open_manipulator_x_description/meshes"/>
+    <xacro:property name="link1_length" value="0.06"/>
     <xacro:if value="${parent_link != ''}">
       <joint name="${prefix}${parent_link}_to_link1" type="fixed">
@@ -17,8 +18,8 @@
     <link name="${prefix}link1">
       <visual>
-        <origin xyz="0 0 0.03" rpy="0 0 0"/>
+        <origin xyz="0 0 ${link1_length/2}" rpy="0 0 0"/>
         <geometry>
           <!-- We use custom cylinder -->
-          <cylinder radius="0.035" length="0.065" />
+          <cylinder radius="0.035" length="${link1_length}" />
           <!-- <mesh filename="${meshes_dir}/link1.stl" scale="0.001 0.001 0.001"/> -->
         </geometry>
@@ -26,8 +27,8 @@
       </visual>
       <collision>
-        <origin xyz="0 0 0.03" rpy="0 0 0"/>
+        <origin xyz="0 0 ${link1_length/2}" rpy="0 0 0"/>
         <geometry>
           <!-- We use custom cylinder -->
-          <cylinder radius="0.035" length="0.065" />
+          <cylinder radius="0.035" length="${link1_length}" />
           <!-- <mesh filename="${meshes_dir}/link1.stl" scale="0.001 0.001 0.001"/> -->
         </geometry>
@@ -45,5 +46,5 @@
       <child link="${prefix}link2"/>
       <!-- Fix origin on custom cylinder -->
-      <origin xyz="0.0 0.0 0.045" rpy="0 0 0"/>
+      <origin xyz="0.0 0.0 0.017" rpy="0 0 0"/>
       <axis xyz="0 0 1"/>
       <limit velocity="4.8" effort="1" lower="${-pi}" upper="${pi}" />
@@ -52,5 +53,5 @@
     <link name="${prefix}link2">
       <visual>
-        <origin xyz="0 0 0" rpy="0 0 0"/>
+        <origin xyz="0 0 0.019" rpy="0 0 0"/>
         <geometry>
           <mesh filename="${meshes_dir}/link2.stl" scale="0.001 0.001 0.001"/>
@@ -59,5 +60,5 @@
       </visual>
       <collision>
-        <origin xyz="0 0 0" rpy="0 0 0"/>
+        <origin xyz="0 0 0.019" rpy="0 0 0"/>
         <geometry>
           <mesh filename="${meshes_dir}/link2.stl" scale="0.001 0.001 0.001"/>

Commit message: General fixes to open manipulator

File: open_manipulator_x_description/urdf/body.xacro (robot description, xacro)
@@ -48,5 +48,5 @@
       <origin xyz="0.0 0.0 0.017" rpy="0 0 0"/>
       <axis xyz="0 0 1"/>
-      <limit velocity="4.8" effort="1" lower="${-pi}" upper="${pi}" />
+      <limit velocity="4.8" effort="1" lower="${-5/4*pi}" upper="${3/4*pi}" />
       <dynamics damping="0.1"/>
     </joint>
@@ -78,5 +78,5 @@
       <origin xyz="0.0 0.0 0.0595" rpy="0 0 0"/>
       <axis xyz="0 1 0"/>
-      <limit velocity="4.8" effort="1" lower="${-1.5}" upper="${1.5}" />
+      <limit velocity="4.8" effort="1" lower="${-pi}" upper="${pi}" />
       <dynamics damping="0.1"/>
     </joint>
