Commit message: Great update Open Manipulation for ROSbot XL Manipulation

File: open_manipulator_x_description/urdf/body.xacro (robot description, xacro)
@@ -8,6 +8,7 @@
                     prefix:=''">
     <xacro:property name="meshes_dir" value="package://open_manipulator_x_description/meshes"/>
+    <xacro:property name="link1_length" value="0.06"/>
     <xacro:if value="${parent_link != ''}">
-      <joint name="${prefix}${parent_link}_joint" type="fixed">
+      <joint name="${prefix}${parent_link}_to_link1" type="fixed">
         <origin xyz="${xyz}" rpy="${rpy}" />
         <parent link="${parent_link}"/>
@@ -17,8 +18,8 @@
     <link name="${prefix}link1">
       <visual>
-        <origin xyz="0 0 0.03" rpy="0 0 0"/>
+        <origin xyz="0 0 ${link1_length/2}" rpy="0 0 0"/>
         <geometry>
           <!-- We use custom cylinder -->
-          <cylinder radius="0.035" length="0.065" />
+          <cylinder radius="0.035" length="${link1_length}" />
           <!-- <mesh filename="${meshes_dir}/link1.stl" scale="0.001 0.001 0.001"/> -->
         </geometry>
@@ -26,8 +27,8 @@
       </visual>
       <collision>
-        <origin xyz="0 0 0.03" rpy="0 0 0"/>
+        <origin xyz="0 0 ${link1_length/2}" rpy="0 0 0"/>
         <geometry>
           <!-- We use custom cylinder -->
-          <cylinder radius="0.035" length="0.065" />
+          <cylinder radius="0.035" length="${link1_length}" />
           <!-- <mesh filename="${meshes_dir}/link1.stl" scale="0.001 0.001 0.001"/> -->
         </geometry>
@@ -45,12 +46,12 @@
       <child link="${prefix}link2"/>
       <!-- Fix origin on custom cylinder -->
-      <origin xyz="0.0 0.0 0.045" rpy="0 0 0"/>
+      <origin xyz="0.0 0.0 0.017" rpy="0 0 0"/>
       <axis xyz="0 0 1"/>
-      <limit velocity="4.8" effort="1" lower="${-pi}" upper="${pi}" />
+      <limit velocity="4.8" effort="1" lower="${-5/4*pi}" upper="${3/4*pi}" />
       <dynamics damping="0.1"/>
     </joint>
     <link name="${prefix}link2">
       <visual>
-        <origin xyz="0 0 0" rpy="0 0 0"/>
+        <origin xyz="0 0 0.019" rpy="0 0 0"/>
         <geometry>
           <mesh filename="${meshes_dir}/link2.stl" scale="0.001 0.001 0.001"/>
@@ -59,5 +60,5 @@
       </visual>
       <collision>
-        <origin xyz="0 0 0" rpy="0 0 0"/>
+        <origin xyz="0 0 0.019" rpy="0 0 0"/>
         <geometry>
           <mesh filename="${meshes_dir}/link2.stl" scale="0.001 0.001 0.001"/>
@@ -77,5 +78,5 @@
       <origin xyz="0.0 0.0 0.0595" rpy="0 0 0"/>
       <axis xyz="0 1 0"/>
-      <limit velocity="4.8" effort="1" lower="${-1.5}" upper="${1.5}" />
+      <limit velocity="4.8" effort="1" lower="${-pi/2}" upper="${pi/2}" />
       <dynamics damping="0.1"/>
     </joint>

File: open_manipulator_x_description/urdf/ros2_control.xacro (robot description, xacro)
@@ -6,5 +6,5 @@
       <xacro:if value="$(arg use_sim)">
         <hardware>
-          <plugin>ign_ros2_control/IgnitionSystem</plugin>
+          <plugin>gz_ros2_control/GazeboSimSystem</plugin>
         </hardware>
       </xacro:if>
@@ -22,5 +22,5 @@
             <param name="error_timeout_ms">500</param>
             <param name="dynamixel_model_folder">/param/dxl_model</param>
-            <param name="number_of_joints">5</param>
+            <param name="number_of_joints">6</param>
             <param name="number_of_transmissions">5</param>
             <param name="transmission_to_joint_matrix">
@@ -29,12 +29,13 @@
               0, 0, 1, 0, 0,
               0, 0, 0, 1, 0,
-              0, 0, 0, 0, 1
+              0, 0, 0, 0, 1,
+              0, 0, 0, 0, 0
             </param>
             <param name="joint_to_transmission_matrix">
-              1, 0, 0, 0, 0,
-              0, 1, 0, 0, 0,
-              0, 0, 1, 0, 0,
-              0, 0, 0, 1, 0,
-              0, 0, 0, 0, 1
+              1, 0, 0, 0, 0, 0,
+              0, 1, 0, 0, 0, 0,
+              0, 0, 1, 0, 0, 0,
+              0, 0, 0, 1, 0, 0,
+              0, 0, 0, 0, 1, 0
             </param>
             <param name="ros_update_freq">200</param>
@@ -86,4 +87,10 @@
         <state_interface name="effort"/>
       </joint>
+      <joint name="${prefix}gripper_right_joint">
+        <command_interface name="position"/>
+        <state_interface name="position"/>
+        <state_interface name="velocity"/>
+        <state_interface name="effort"/>
+      </joint>
       <gpio name="dxl1">
         <param name="type">dxl</param>
@@ -101,4 +108,5 @@
         <param name="Profile Acceleration">50</param>
         <param name="Drive Mode">0</param>
+        <param name="Return Delay Time">0</param>
       </gpio>
       <gpio name="dxl2">
@@ -117,4 +125,5 @@
         <param name="Profile Acceleration">50</param>
         <param name="Drive Mode">0</param>
+        <param name="Return Delay Time">0</param>
       </gpio>
       <gpio name="dxl3">
@@ -133,4 +142,5 @@
         <param name="Profile Acceleration">50</param>
         <param name="Drive Mode">0</param>
+        <param name="Return Delay Time">0</param>
       </gpio>
       <gpio name="dxl4">
@@ -149,4 +159,5 @@
         <param name="Profile Acceleration">50</param>
         <param name="Drive Mode">0</param>
+        <param name="Return Delay Time">0</param>
       </gpio>
       <gpio name="dxl5">
@@ -159,4 +170,5 @@
         <state_interface name="Torque Enable"/>
         <state_interface name="Present Input Voltage"/>
+        <param name="Return Delay Time">0</param>
       </gpio>
     </ros2_control>

Commit message: Improve gamepad control

File: open_manipulator_x_description/urdf/body.xacro (robot description, xacro)
@@ -48,5 +48,5 @@
       <origin xyz="0.0 0.0 0.017" rpy="0 0 0"/>
       <axis xyz="0 0 1"/>
-      <limit velocity="4.8" effort="1" lower="${-5/4*pi}" upper="${3/4*pi}" />
+      <limit velocity="4.8" effort="1" lower="${-4/5*pi}" upper="${pi}" />
       <dynamics damping="0.1"/>
     </joint>

Commit message: Use official open_manipulator_description package

File: open_manipulator_x_description/urdf/body.xacro (robot description, xacro)
@@ -7,5 +7,5 @@
                     namespace:=''
                     prefix:=''">
-    <xacro:property name="meshes_dir" value="package://open_manipulator_x_description/meshes"/>
+    <xacro:property name="meshes_dir" value="package://open_manipulator_description/meshes/open_manipulator_x"/>
     <xacro:property name="link1_length" value="0.06"/>
     <xacro:if value="${parent_link != ''}">

File: open_manipulator_x_description/urdf/open_manipulator_x_macro.xacro (robot description, xacro)
@@ -15,7 +15,6 @@
     <!-- INCLUDE ROBOT MACRO -->
     <xacro:include filename="$(find open_manipulator_x_description)/urdf/body.xacro" ns="body"/>
-    <xacro:include filename="$(find open_manipulator_x_description)/urdf/materials.xacro" />
-    <xacro:include filename="$(find open_manipulator_x_description)/urdf/gazebo.xacro"  ns="gazebo" />
-    <xacro:include filename="$(find open_manipulator_x_description)/urdf/ros2_control.xacro" ns="ros2_control" />
+    <xacro:include filename="$(find open_manipulator_description)/gazebo/open_manipulator_x.gazebo.xacro"  ns="gazebo" />
+    <xacro:include filename="$(find open_manipulator_description)/ros2_control/open_manipulator_x_position.ros2_control.xacro" ns="ros2_control" />
     <!-- BODY -->
     <xacro:body.open_manipulator_x
@@ -34,5 +33,5 @@
     <!-- GAZEBO PLUGINS -->
     <xacro:if value="${use_sim}">
-      <xacro:gazebo.gz_open_manipulator_x_system prefix="${prefix}" />
+      <xacro:gazebo.open_manipulator_x_gazebo prefix="${prefix}" />
     </xacro:if>
   </xacro:macro>

Commit message: Fix colors

File: open_manipulator_x_description/urdf/body.xacro (robot description, xacro)
@@ -24,5 +24,7 @@
           <!-- <mesh filename="${meshes_dir}/link1.stl" scale="0.001 0.001 0.001"/> -->
         </geometry>
-        <material name="grey"/>
+        <material name="grey">
+          <color rgba="0.2 0.2 0.2 1"/>
+        </material>
       </visual>
       <collision>
@@ -57,5 +59,7 @@
           <mesh filename="${meshes_dir}/link2.stl" scale="0.001 0.001 0.001"/>
         </geometry>
-        <material name="grey"/>
+        <material name="grey">
+          <color rgba="0.2 0.2 0.2 1"/>
+        </material>
       </visual>
       <collision>
@@ -87,5 +91,7 @@
           <mesh filename="${meshes_dir}/link3.stl" scale="0.001 0.001 0.001"/>
         </geometry>
-        <material name="grey"/>
+        <material name="grey">
+          <color rgba="0.2 0.2 0.2 1"/>
+        </material>
       </visual>
       <collision>
@@ -117,5 +123,7 @@
           <mesh filename="${meshes_dir}/link4.stl" scale="0.001 0.001 0.001"/>
         </geometry>
-        <material name="grey"/>
+        <material name="grey">
+          <color rgba="0.2 0.2 0.2 1"/>
+        </material>
       </visual>
       <collision>
@@ -147,5 +155,7 @@
           <mesh filename="${meshes_dir}/link5.stl" scale="0.001 0.001 0.001"/>
         </geometry>
-        <material name="grey"/>
+        <material name="grey">
+          <color rgba="0.2 0.2 0.2 1"/>
+        </material>
       </visual>
       <collision>
@@ -177,5 +187,7 @@
           <mesh filename="${meshes_dir}/gripper_left_palm.stl" scale="0.001 0.001 0.001"/>
         </geometry>
-        <material name="grey"/>
+        <material name="grey">
+          <color rgba="0.2 0.2 0.2 1"/>
+        </material>
       </visual>
       <collision>
@@ -208,5 +220,7 @@
           <mesh filename="${meshes_dir}/gripper_right_palm.stl" scale="0.001 0.001 0.001"/>
         </geometry>
-        <material name="grey"/>
+        <material name="grey">
+          <color rgba="0.2 0.2 0.2 1"/>
+        </material>
       </visual>
       <collision>

File: open_manipulator_x_description/urdf/open_manipulator_x_macro.xacro (robot description, xacro)
@@ -15,5 +15,5 @@
     <!-- INCLUDE ROBOT MACRO -->
     <xacro:include filename="$(find open_manipulator_x_description)/urdf/body.xacro" ns="body"/>
-    <xacro:include filename="$(find open_manipulator_x_description)/urdf/materials.xacro" />
+    <!-- <xacro:include filename="$(find open_manipulator_x_description)/urdf/materials.xacro" /> -->
     <xacro:include filename="$(find open_manipulator_description)/gazebo/open_manipulator_x.gazebo.xacro"  ns="gazebo" />
     <xacro:include filename="$(find open_manipulator_description)/ros2_control/open_manipulator_x_position.ros2_control.xacro" ns="ros2_control" />

Commit message: Use official open_manipulator_description package (#14)

File: open_manipulator_x_description/urdf/body.xacro (robot description, xacro)
@@ -7,5 +7,5 @@
                     namespace:=''
                     prefix:=''">
-    <xacro:property name="meshes_dir" value="package://open_manipulator_x_description/meshes"/>
+    <xacro:property name="meshes_dir" value="package://open_manipulator_description/meshes/open_manipulator_x"/>
     <xacro:property name="link1_length" value="0.06"/>
     <xacro:if value="${parent_link != ''}">
@@ -24,5 +24,7 @@
           <!-- <mesh filename="${meshes_dir}/link1.stl" scale="0.001 0.001 0.001"/> -->
         </geometry>
-        <material name="grey"/>
+        <material name="grey">
+          <color rgba="0.2 0.2 0.2 1"/>
+        </material>
       </visual>
       <collision>
@@ -57,5 +59,7 @@
           <mesh filename="${meshes_dir}/link2.stl" scale="0.001 0.001 0.001"/>
         </geometry>
-        <material name="grey"/>
+        <material name="grey">
+          <color rgba="0.2 0.2 0.2 1"/>
+        </material>
       </visual>
       <collision>
@@ -87,5 +91,7 @@
           <mesh filename="${meshes_dir}/link3.stl" scale="0.001 0.001 0.001"/>
         </geometry>
-        <material name="grey"/>
+        <material name="grey">
+          <color rgba="0.2 0.2 0.2 1"/>
+        </material>
       </visual>
       <collision>
@@ -117,5 +123,7 @@
           <mesh filename="${meshes_dir}/link4.stl" scale="0.001 0.001 0.001"/>
         </geometry>
-        <material name="grey"/>
+        <material name="grey">
+          <color rgba="0.2 0.2 0.2 1"/>
+        </material>
       </visual>
       <collision>
@@ -147,5 +155,7 @@
           <mesh filename="${meshes_dir}/link5.stl" scale="0.001 0.001 0.001"/>
         </geometry>
-        <material name="grey"/>
+        <material name="grey">
+          <color rgba="0.2 0.2 0.2 1"/>
+        </material>
       </visual>
       <collision>
@@ -177,5 +187,7 @@
           <mesh filename="${meshes_dir}/gripper_left_palm.stl" scale="0.001 0.001 0.001"/>
         </geometry>
-        <material name="grey"/>
+        <material name="grey">
+          <color rgba="0.2 0.2 0.2 1"/>
+        </material>
       </visual>
       <collision>
@@ -208,5 +220,7 @@
           <mesh filename="${meshes_dir}/gripper_right_palm.stl" scale="0.001 0.001 0.001"/>
         </geometry>
-        <material name="grey"/>
+        <material name="grey">
+          <color rgba="0.2 0.2 0.2 1"/>
+        </material>
       </visual>
       <collision>

Commit message: Use mesh form official ROS 2 package

File: open_manipulator_x_description/urdf/body.xacro (robot description, xacro)
@@ -24,5 +24,7 @@
           <!-- <mesh filename="${meshes_dir}/link1.stl" scale="0.001 0.001 0.001"/> -->
         </geometry>
-        <material name="grey"/>
+        <material name="grey">
+          <color rgba="0.2 0.2 0.2 1"/>
+        </material>
       </visual>
       <collision>
@@ -57,5 +59,7 @@
           <mesh filename="${meshes_dir}/link2.stl" scale="0.001 0.001 0.001"/>
         </geometry>
-        <material name="grey"/>
+        <material name="grey">
+          <color rgba="0.2 0.2 0.2 1"/>
+        </material>
       </visual>
       <collision>
@@ -87,5 +91,7 @@
           <mesh filename="${meshes_dir}/link3.stl" scale="0.001 0.001 0.001"/>
         </geometry>
-        <material name="grey"/>
+        <material name="grey">
+          <color rgba="0.2 0.2 0.2 1"/>
+        </material>
       </visual>
       <collision>
@@ -117,5 +123,7 @@
           <mesh filename="${meshes_dir}/link4.stl" scale="0.001 0.001 0.001"/>
         </geometry>
-        <material name="grey"/>
+        <material name="grey">
+          <color rgba="0.2 0.2 0.2 1"/>
+        </material>
       </visual>
       <collision>
@@ -147,5 +155,7 @@
           <mesh filename="${meshes_dir}/link5.stl" scale="0.001 0.001 0.001"/>
         </geometry>
-        <material name="grey"/>
+        <material name="grey">
+          <color rgba="0.2 0.2 0.2 1"/>
+        </material>
       </visual>
       <collision>
@@ -177,5 +187,7 @@
           <mesh filename="${meshes_dir}/gripper_left_palm.stl" scale="0.001 0.001 0.001"/>
         </geometry>
-        <material name="grey"/>
+        <material name="grey">
+          <color rgba="0.2 0.2 0.2 1"/>
+        </material>
       </visual>
       <collision>
@@ -208,5 +220,7 @@
           <mesh filename="${meshes_dir}/gripper_right_palm.stl" scale="0.001 0.001 0.001"/>
         </geometry>
-        <material name="grey"/>
+        <material name="grey">
+          <color rgba="0.2 0.2 0.2 1"/>
+        </material>
       </visual>
       <collision>

File: open_manipulator_x_description/urdf/open_manipulator_x_macro.xacro (robot description, xacro)
@@ -15,5 +15,4 @@
     <!-- INCLUDE ROBOT MACRO -->
     <xacro:include filename="$(find open_manipulator_x_description)/urdf/body.xacro" ns="body"/>
-    <xacro:include filename="$(find open_manipulator_x_description)/urdf/materials.xacro" />
     <xacro:include filename="$(find open_manipulator_x_description)/urdf/gazebo.xacro"  ns="gazebo" />
     <xacro:include filename="$(find open_manipulator_x_description)/urdf/ros2_control.xacro" ns="ros2_control" />
